File: torpedo_pcbs/PCB_main_board/PCB_main_board.kicad_sch (KiCad schematic)
At the start: 52 parts, among them IC1 ESP-PSRAM64H, IC2 TMUX4052PWRQ1, IC3 ESP32-S3-WROOM-1U-N8R8, J1 5051102491, J10 Micro_SD_Card, J2 USB_C_Receptacle_USB2.0_16P, J3 Conn_01x05, J5 5051102491, J6 5051102491, Q2 BC817, Q3 BC817, Q4 PMOS, U1 ICM-20948, U2 CH340C, U3 ESP32-WROOM-32D, U5 XC6206PxxxMR, U6 XC6206PxxxMR, U7 ESP-PSRAM32, U8 ESP32-S3-WROOM-1

Commit message: psram already in esp32, minor updates
Parts:
- removed C1, C2: 0.1 μF, symbol Device:C
- removed C16: 1μF, symbol Device:C
- removed IC1: ESP-PSRAM64H, SOIC127P600X175-8N, symbol SamacSys_Parts:ESP-PSRAM64H
- removed Q3: BC817, Package_TO_SOT_SMD:SOT-23, symbol Transistor_BJT:BC817
- removed R17: 10k, symbol Device:R
- removed U2: CH340C, Package_SO:SOIC-16_3.9x9.9mm_P1.27mm, symbol Interface_USB:CH340C
- removed U7: ESP-PSRAM32, Package_SO:SOIC-8_3.9x4.9mm_P1.27mm, symbol Memory_RAM:ESP-PSRAM32
- added Q1: BC817, Package_TO_SOT_SMD:SOT-23, symbol Transistor_BJT:BC817
- added R5: 10k, symbol Device:R
- R3: value 10k -> 47k
Connections:
- net +3.3V: now also R3.2
- net ESP_EN: now also IC3.16 (IO46), IC3.3 (EN), Q2.3 (C)
- net ESP_IO0: now also IC3.27 (IO0), Q1.3 (C); no longer Q2.3 (C)
- net GND: now also U1.9 (SDO/AD0)
- net HS2_DATA2: now also R3.1
- net RX: no longer IC3.36 (RXD0)
- net TX: no longer IC3.37 (TXD0)
- net at Q2.1 (B): now also R5.1; no longer R3.1
- net at R4.1: now also Q1.1 (B)
- net at R4.2: no longer Q2.2 (E)
- net D-: now reaches IC3.13 (IO19)
- net D-: now also J2.A7 (D-), J2.B7 (D-)
- net D+: now reaches IC3.14 (IO20)
- net D+: now also J2.A6 (D+), J2.B6 (D+)
- net EN: no longer names the net of C15.2, R12.2
- net EN: no longer IC3.3 (EN)
- new net: Q1.2 (E), R5.2
- no-connect marks 23 -> 18
Other:
- note added: "Power/Flash"
- note added: "This was labeled as NC, but <---- still create a pad for a resistor just in case"
- note added: "What needs to be connected? - (i guess anywhere) Cameras - (anywhere) Cam switch - (anywhere) I2C - SD card (DONE)"
- note removed: "I have no clue how to connect this"
- note removed: "Power/Batteries"
- note removed: "What needs to be connected? - (i guess anywhere) Cameras - (anywhere) Cam switch - (anywhere) I2C - SD card (DONE) - PSRAM"
- note removed: "Working datasheet link: https://cdn-shop.adafruit.com/product-files/4677/4677_esp-psram64_esp-psram64h_datasheet_en.pdf"
- moved on the sheet: C14, C15, IC3, J2, R1, R12, R2

Commit message: daugther board started
Parts:
- removed IC3: ESP32-S3-WROOM-1U-N8R8, ESP32S3WROOM1UN8R8, symbol SamacSys_Parts:ESP32-S3-WROOM-1U-N8R8
- removed J10: Micro_SD_Card, symbol Connector:Micro_SD_Card
- removed J2: USB_C_Receptacle_USB2.0_16P, Connector_USB:USB_C_Receptacle_GCT_USB4085, symbol Connector:USB_C_Receptacle_USB2.0_16P
- removed Q1, Q2: BC817, Package_TO_SOT_SMD:SOT-23, symbol Transistor_BJT:BC817
- removed Q4: PMOS, symbol Simulation_SPICE:PMOS
- removed R11, R12, R5: 10k, symbol Device:R
- removed R7: 1k, symbol Device:R
- removed U3: ESP32-WROOM-32D, RF_Module:ESP32-WROOM-32D, symbol RF_Module:ESP32-WROOM-32D
- removed U8: ESP32-S3-WROOM-1, PCM_Espressif:ESP32-S3-WROOM-1, symbol PCM_Espressif:ESP32-S3-WROOM-1
- added C1: 22μF, Capacitor_SMD:C_0805_2012Metric_Pad1.18x1.45mm_HandSolder, symbol Device:C
- added C2: 1μF, Capacitor_SMD:C_0805_2012Metric_Pad1.18x1.45mm_HandSolder, symbol Device:C
- added D1: RCLAMP7522T.TNT, samacsys_parts:RCLAMP7522TTNT, symbol SamacSys_Parts:RCLAMP7522T.TNT
- added IC4: ESP32-S3-WROOM-1U-N8R8, PCM_Espressif:ESP32-S3-WROOM-1U, symbol SamacSys_Parts:ESP32-S3-WROOM-1U-N8R8
- added J2: MSD-4-A, samacsys_parts:MSD4A, symbol SamacSys_Parts:MSD-4-A
- added J4: Conn_01x02, Connector_PinSocket_2.00mm:PinSocket_1x02_P2.00mm_Vertical, symbol Connector_Generic:Conn_01x02
- added J7: GSB1C4621DS1HR, Connector_USB:12402054M611A, symbol SamacSys_Parts:GSB1C4621DS1HR
- added J9: Conn_01x03, Connector_PinSocket_2.00mm:PinSocket_1x03_P2.00mm_Vertical, symbol Connector_Generic:Conn_01x03
- added R14, R17: 5.1k, Capacitor_SMD:C_0805_2012Metric_Pad1.18x1.45mm_HandSolder, symbol Device:R
- added S1, S3: CS1213AGF260, CS1213AGF260, symbol SamacSys_Parts:CS1213AGF260
- C10, C11, C12, C13, C14, C15, C17, C3, C4, C5, C6, C7, C8, C9, R10, R13, R15, R16, R18, R3, R8, R9: footprint (none) -> Capacitor_SMD:C_0805_2012Metric_Pad1.18x1.45mm_HandSolder
- IC2: footprint SOP65P640X120-16N -> samacsys_parts:SOP65P640X120-16N
- J1, J5, J6: footprint 5051102491 -> samacsys_parts:5051102491
- J3: footprint (none) -> Connector_PinHeader_2.54mm:PinHeader_1x05_P2.54mm_Vertical
- R1: value 5.1k -> 10k; footprint (none) -> Capacitor_SMD:C_0805_2012Metric_Pad1.18x1.45mm_HandSolder
- R2: value 5.1k -> 2.2k; footprint (none) -> Capacitor_SMD:C_0805_2012Metric_Pad1.18x1.45mm_HandSolder
- R4: value 10k -> 2.2k; footprint (none) -> Capacitor_SMD:C_0805_2012Metric_Pad1.18x1.45mm_HandSolder
- R6: value 10k -> 1k; footprint (none) -> Capacitor_SMD:C_0805_2012Metric_Pad1.18x1.45mm_HandSolder
Connections:
- net SCI_XCLK is gone; now on net CSI_PWDN: IC2.13 (DA)
- net +3.3V: now also R1.1, R2.1, R4.1, U5.3 (VI), U6.3 (VI), C1.2, IC4.2 (3V3), J2.4 (VDD)
- net CAM_SWITCH0: now also IC4.34 (IO41)
- net CAM_SWITCH1: now also IC4.35 (IO42)
- net CSI_D0: now also IC4.20 (IO12)
- net CSI_D1: now also IC4.18 (IO10)
- net CSI_D2: now also IC4.17 (IO9)
- net CSI_D3: now also IC4.19 (IO11)
- net CSI_D4: now also IC4.21 (IO13)
- net CSI_D5: now also IC4.22 (IO14)
- net CSI_D6: now also IC4.23 (IO21)
- net CSI_D7: now also IC4.24 (IO47)
- net CSI_HSYNC: now also IC4.25 (IO48)
- net CSI_PCLK: now also IC4.12 (IO8)
- net CSI_PWDN: now also IC4.33 (IO40)
- net CSI_VSYNC: now also IC4.26 (IO45)
- net D+: now also D1.3 (I2C-SDC), IC4.14 (IO20), J7.A6 (DP1), J7.B6 (DP2)
- net D-: now also D1.4 (I2C-SDA), IC4.13 (IO19), J7.A7 (DN1), J7.B7 (DN2)
- net ESP_EN: now also C15.1, R1.2, C2.2, IC4.16 (IO46), IC4.3 (EN), S3.1 (NO)
- net GND: now also C15.2, C1.1, C2.1, D1.5 (RESET), IC4.1 (GND_1), IC4.40 (GND_2), IC4.41 (GND_3), IC4.42 (GND_4), IC4.43 (GND_5), IC4.44 (GND_6), IC4.45 (GND_7), IC4.46 (GND_8), IC4.47 (GND_9), IC4.48 (GND_10), IC4.49 (GND_11), J2.6 (VSS), J2.G1 (GND_1), J2.G2 (GND_2), J2.G3 (GND_3), J2.G4 (GND_4), J7.A1 (GND_1), J7.A12 (GND_2), J7.MH1, J7.MH2, J7.MH3, J7.MH4, R14.1, R17.1, S1.2 (COM), S3.2 (COM); no longer C15.1, R1.1, R2.1
- net HS2_CLK: now also IC4.8 (IO15), J2.5 (CLK)
- net HS2_CMD: now also IC4.4 (IO4), J2.3 (CMD)
- net HS2_DATA0: now also IC4.9 (IO16), J2.7 (DAT0)
- net HS2_DATA1: now also IC4.10 (IO17), J2.8 (DAT1)
- net HS2_DATA2: now also IC4.38 (IO2), J2.1 (DAT2)
- net HS2_DATA3: now also IC4.39 (IO1), J2.2 (CD/DAT3)
- net PWDN_CAM1: now also IC2.12 (S0A); no longer IC2.1 (S0B)
- net PWDN_CAM2: now also IC2.14 (S1A); no longer IC2.5 (S1B)
- net PWDN_CAM3: now also IC2.15 (S2A); no longer IC2.2 (S2B)
- net SCL: now also J3.4 (Pin_4), R4.2, IC4.7 (IO7); no longer J3.5 (Pin_5)
- net SDA: now also J3.5 (Pin_5), R2.2, IC4.6 (IO6); no longer J3.4 (Pin_4)
- net TWI_SCK: now also IC4.31 (IO38)
- net TWI_SDA: now also IC4.32 (IO39)
- net VBUS: now also D1.1 (GND), J7.A4 (VBUS_1), J7.A9 (VBUS_2)
- net XCLK_CAM1: now also IC2.1 (S0B); no longer IC2.12 (S0A)
- net XCLK_CAM2: now also IC2.5 (S1B); no longer IC2.14 (S1A)
- net XCLK_CAM3: now also IC2.2 (S2B); no longer IC2.15 (S2A)
- net SCI_PWDN renamed BOOT
- net BOOT: now also IC4.27 (IO0), S1.1 (NO)
- new net: J7.B5 (CC2), R14.2
- new net: J7.A5 (CC1), R17.2
- new net JTAG/extra_IO3: IC4.15 (IO3), J4.1 (Pin_1)
- new net extra_IO18: IC4.11 (IO18), J4.2 (Pin_2)
- new net extra_IO35: IC4.28 (IO35), J9.3 (Pin_3)
- new net extra_IO36: IC4.29 (IO36), J9.2 (Pin_2)
- new net extra_IO37: IC4.30 (IO37), J9.1 (Pin_1)
- new net extra_IO5: IC4.5 (IO5)
- no-connect marks 18 -> 19
Other:
- note removed: "Missing gpio:"
- note removed: "What needs to be connected? - (i guess anywhere) Cameras - (anywhere) Cam switch - (anywhere) I2C - SD card (DONE)"
- moved on the sheet: C14, C7
