File: torpedo_pcbs/PCB_battery_motor_board/PCB_battery_motor_board.kicad_pcb (KiCad board)
At the start: 2 copper layers, 23.7 x 17.8 mm, 48 parts, among them IC2 BQ25601RTWR, IC3 DRV8235RTER, IC4 DRV8235RTER, IC5 DRV8235RTER, IC6 DRV8235RTER, J1 Conn_01x01, J10 Conn_01x05, J3 Conn_01x02, J4 Conn_01x01, J5 Conn_01x02, J6 Conn_01x02, J7 Conn_01x04, J8 Conn_01x02, J9 Conn_01x02, U1 AMS1117-3.3

Commit message: finished saving
Parts:
- moved J6 0.43 mm to (109.0, 86.8)
Changed lines of the file:
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@@
 		)
 		(model "${KICAD8_3DMODEL_DIR}/Connector_PinSocket_2.00mm.3dshapes/PinSocket_1x02_P2.00mm_Vertical.wrl"
+			(hide yes)
 			(offset
 				(xyz 0 0 0)
@@
 		)
 		(model "${KICAD8_3DMODEL_DIR}/Connector_PinSocket_2.00mm.3dshapes/PinSocket_1x02_P2.00mm_Vertical.wrl"
+			(hide yes)
 			(offset
 				(xyz 0 0 0)
@@
 		)
 		(model "${KICAD8_3DMODEL_DIR}/Connector_PinSocket_2.00mm.3dshapes/PinSocket_1x02_P2.00mm_Vertical.wrl"
+			(hide yes)
 			(offset
 				(xyz 0 0 0)
@@
 		)
 		(model "${KICAD8_3DMODEL_DIR}/Connector_PinSocket_2.00mm.3dshapes/PinSocket_1x05_P2.00mm_Vertical.wrl"
+			(hide yes)
 			(offset
 				(xyz 0 0 0)
@@
 	(footprint "Connector_PinSocket_2.00mm:PinSocket_1x02_P2.00mm_Vertical"
 		(layer "F.Cu")
-		(at 108.6 86.875 90)
+		(at 109.025 86.825 90)
 		(descr "Through hole straight socket strip, 1x02, 2.00mm pitch, single row (from Kicad 4.0.7), script generated")
 		(tags "Through hole socket strip THT 1x02 2.00mm single row")
@@
 		)
 		(model "${KICAD8_3DMODEL_DIR}/Connector_PinSocket_2.00mm.3dshapes/PinSocket_1x02_P2.00mm_Vertical.wrl"
+			(hide yes)
 			(offset
 				(xyz 0 0 0)
@@
 		)
 		(model "${KICAD8_3DMODEL_DIR}/Connector_PinSocket_2.00mm.3dshapes/PinSocket_1x04_P2.00mm_Vertical.wrl"
+			(hide yes)
 			(offset
 				(xyz 0 0 0)
@@
 		)
 		(model "${KICAD8_3DMODEL_DIR}/Connector_PinSocket_2.00mm.3dshapes/PinSocket_1x02_P2.00mm_Vertical.wrl"
+			(hide yes)
 			(offset
 				(xyz 0 0 0)

Commit message: daughter board updates
Parts:
- added R19: 0, Resistor_SMD:R_0805_2012Metric_Pad1.20x1.40mm_HandSolder, F.Cu at (111.5, 104.5)
- added R20: 0, Resistor_SMD:R_0805_2012Metric_Pad1.20x1.40mm_HandSolder, F.Cu at (136.8, 104.5)
- added R4: 0, Resistor_SMD:R_0805_2012Metric_Pad1.20x1.40mm_HandSolder, F.Cu at (129.0, 104.5)
- added R5: 0, Resistor_SMD:R_0805_2012Metric_Pad1.20x1.40mm_HandSolder, F.Cu at (120.0, 104.5)
- C1, C2, C5, D2, D3, IC2, J9, L2, R6, R7, U1: moved to B.Cu
- J10: footprint Connector_PinSocket_2.00mm:PinSocket_1x05_P2.00mm_Vertical -> SamacSys_Parts:S5BPHKSLFSN
- moved R2 81.8 mm to (127.8, 97.2), turned to -90 degrees
- moved R6 73.5 mm to (119.5, 101.0), turned to -90 degrees
- moved R1 73.2 mm to (118.8, 97.8), turned to 90 degrees
- moved R7 66.2 mm to (112.2, 103.0), turned to 180 degrees
- moved R17 65.2 mm to (141.8, 98.5), turned to -90 degrees
- moved R23 65.2 mm to (141.8, 102.5), turned to -90 degrees
- moved C1 64.4 mm to (119.5, 97.0), turned to -90 degrees
- moved R3 63.2 mm to (109.0, 101.5), turned to 90 degrees
- moved R9 58.7 mm to (109.0, 97.5), turned to 90 degrees
- moved C5 58.2 mm to (112.9, 88.3), turned to -90 degrees
- moved C9 58.2 mm to (138.7, 97.2), turned to 180 degrees
- moved R18 58.1 mm to (134.2, 102.5), turned to -90 degrees
- moved R14 58.0 mm to (134.3, 98.5), turned to -90 degrees
- moved IC6 56.9 mm to (138.5, 100.5), turned to 180 degrees
- moved C2 52.1 mm to (107.5, 97.0), turned to -90 degrees
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Connections:
- C1 pad 1: /SYS_PWR -> SYS_PWR
- C3 pad 1: /DC Motor Driver - Rudder-left/SYS_PWR -> SYS_PWR
- C4 pad 1: /SYS_PWR -> SYS_PWR
- C5 pad 1: /SYS_PWR -> SYS_PWR
- C6 pad 1: /DC Motor Driver - Rudder-right/SYS_PWR -> SYS_PWR
- C8 pad 1: /DC Motor Driver - Prop/SYS_PWR -> SYS_PWR
- C9 pad 1: /DC Motor Driver - Extra/SYS_PWR -> SYS_PWR
- D2 pad 2: /SYS_PWR -> SYS_PWR
- D3 pad 2: /SYS_PWR -> SYS_PWR
- IC2 pad 15: /SYS_PWR -> SYS_PWR
- IC2 pad 16: /SYS_PWR -> SYS_PWR
- IC3 pad 14: /SDA -> /DC Motor Driver - Rudder-left/SDA
- IC3 pad 16: /DC Motor Driver - Rudder-left/VREF -> VREF
- IC3 pad 5: /DC Motor Driver - Rudder-left/SYS_PWR -> SYS_PWR
- IC4 pad 14: /SDA -> /DC Motor Driver - Prop/SDA
- IC4 pad 16: /DC Motor Driver - Prop/VREF -> VREF
- IC4 pad 5: /DC Motor Driver - Prop/SYS_PWR -> SYS_PWR
- IC5 pad 14: /SDA -> /DC Motor Driver - Rudder-right/SDA
- IC5 pad 16: /DC Motor Driver - Rudder-right/VREF -> VREF
- IC5 pad 5: /DC Motor Driver - Rudder-right/SYS_PWR -> SYS_PWR
- IC6 pad 14: /SDA -> /DC Motor Driver - Extra/SDA
- IC6 pad 16: /DC Motor Driver - Extra/VREF -> VREF
- IC6 pad 5: /DC Motor Driver - Extra/SYS_PWR -> SYS_PWR
- L2 pad 2: /SYS_PWR -> SYS_PWR
- R6 pad 2: /VREF -> VREF
- R7 pad 1: /VREF -> VREF
- U1 pad 3: /SYS_PWR -> SYS_PWR
Routing:
- net /SCL: track 0.00 -> 70.4 mm
- net /SDA: track 0.00 -> 60.8 mm
- net GND: track 0.00 -> 52.6 mm, vias 0 -> 33
- net VREF: track 0.00 -> 30.2 mm, vias 0 -> 4
- net SYS_PWR: track 0.00 -> 23.0 mm, vias 0 -> 7
- net +3.3V: track 0.00 -> 22.8 mm, vias 0 -> 7
- net /DC Motor Driver - Prop/OUT2: track 0.00 -> 19.8 mm
- net /DC Motor Driver - Prop/OUT1: track 0.00 -> 19.4 mm
- net /DC Motor Driver - Rudder-right/OUT2: track 0.00 -> 17.9 mm
- net /DC Motor Driver - Rudder-right/OUT1: track 0.00 -> 17.6 mm
- net /DC Motor Driver - Rudder-left/OUT2: track 0.00 -> 15.0 mm
- net /DC Motor Driver - Rudder-left/OUT1: track 0.00 -> 14.4 mm
- net /DC Motor Driver - Extra/OUT2: track 0.00 -> 14.2 mm
- net /DC Motor Driver - Extra/OUT1: track 0.00 -> 13.5 mm
- net Net-(IC2-BAT_1): track 0.00 -> 9.16 mm
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- added copper zone on B.Cu, net +3.3V
- added copper zone on B.Cu, net /VBUS
- added copper zone on B.Cu, net GND
- added copper zone on F.Cu, net GND
- added copper zone on B.Cu, net Net-(IC2-BAT_1)
- added copper zone on B.Cu, net Net-(IC2-SW_1)
- added copper zone on B.Cu, net SYS_PWR
Other:
- board size 23.7 x 17.8 mm -> 45 x 22 mm
