File: torpedo_pcbs/PCB_battery_motor_board/motor_driver.kicad_sch (KiCad schematic)
At the start: 2 parts, among them IC2 DRV8235RTER

Commit message: daugther board started
Parts:
- added R17: 10k, Resistor_SMD:R_0805_2012Metric_Pad1.20x1.40mm_HandSolder, symbol Device:R
- added R23: ???, Resistor_SMD:R_0805_2012Metric_Pad1.20x1.40mm_HandSolder, symbol Device:R
- C3: renamed from C5; footprint (none) -> Capacitor_SMD:C_0805_2012Metric_Pad1.18x1.45mm_HandSolder
- IC3: renamed from IC2; footprint QFN50P300X300X80-17N-D -> SamacSys_Parts:QFN50P300X300X80-17N-D
Connections:
- net +3.3V: now also IC3.11 (NSLEEP), R17.1; no longer IC3.16 (VREF)
- net GND: now also R23.2
- net SYS_PWR: no longer IC3.11 (NSLEEP)
- net at IC3.4 (NFAULT): now also R17.2
- net IPROPI: no longer names the net of IC3.1 (IPROPI)
- net IPROPI: now also R23.1
- new net VREF: IC3.16 (VREF)
- no-connect marks 5 -> 4

Commit message: daughter board updates
Changed lines of the file:
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@@
 	(wire
 		(pts
-			(xy 40.64 55.88) (xy 40.64 57.15)
+			(xy 40.64 50.8) (xy 40.64 57.15)
 		)
 		(stroke
@@
 	(wire
 		(pts
-			(xy 55.88 55.88) (xy 55.88 62.23)
-		)
-		(stroke
-			(width 0)
-			(type default)
-		)
-	)
-	(wire
-		(pts
-			(xy 40.64 55.88) (xy 55.88 55.88)
+			(xy 55.88 50.8) (xy 55.88 62.23)
+		)
+		(stroke
+			(width 0)
+			(type default)
+		)
+	)
+	(wire
+		(pts
+			(xy 40.64 50.8) (xy 55.88 50.8)
 		)
 		(stroke
@@
 		)
 	)
-	(label "SYS_PWR"
-		(at 49.53 55.88 180)
+	(global_label "SYS_PWR"
+		(shape input)
+		(at 40.64 50.8 180)
 		(fields_autoplaced yes)
 		(effects
@@
 				(size 1.27 1.27)
 			)
-			(justify right bottom)
-		)
-	)
-	(label "VREF"
+			(justify right)
+		)
+		(property "Intersheetrefs" "${INTERSHEET_REFS}"
+			(at 29.1882 50.8 0)
+			(effects
+				(font
+					(size 1.27 1.27)
+				)
+				(justify right)
+				(hide yes)
+			)
+		)
+	)
+	(global_label "VREF"
+		(shape input)
 		(at 100.33 64.77 0)
 		(fields_autoplaced yes)
@@
 				(size 1.27 1.27)
 			)
-			(justify left bottom)
-		)
-	)
+			(justify left)
+		)
+		(property "Intersheetrefs" "${INTERSHEET_REFS}"
+			(at 107.9114 64.77 0)
+			(effects
+				(font
+					(size 1.27 1.27)
+				)
+				(justify left)
+				(hide yes)
+			)
+		)
+	)
