File: Powered_Torpedo_V2.1/Powered_Torpedo_V2.1.kicad_pcb (KiCad board)
At the start: 2 copper layers, 70 x 9.5 mm, 13 parts, among them IC3 AND Gate, IC4 Omnipolar Latch, IC5 Latch, J1 Microfit 3.0, J2 Motor, J3 CAPACITOR #2, J4 CAPACITOR #1, Q1 Mosfet

Commit message: June-1-2025 jlcpcb order
Parts:
- removed the J1 at (165.5, 104.6)
- added G***: LOGO, LOGO, F.Cu at (133.8, 104.8)
- added J4: Microfit 3.0, SamacSys_Parts:436500300, B.Cu at (167.1, 104.6)
- C1: moved to F.Cu
- moved C2 11.9 mm to (114.6, 103.2)
- moved C1 8.91 mm to (103.0, 103.5), turned to 90 degrees
- moved J1 6.00 mm to (139.3, 101.8), turned to -90 degrees
- moved IC1 4.75 mm to (107.0, 103.2)
- moved IC2 4.30 mm to (111.8, 103.3)
- moved J3 4.03 mm to (102.5, 102.8), turned to -90 degrees
- moved IC3 2.25 mm to (118.3, 105.5)
- moved R2 0.75 mm to (111.9, 106.8), turned to 180 degrees
- moved R1 0.51 mm to (107.1, 108.0), turned to 180 degrees
- moved Q1 0.25 mm to (108.0, 103.0)
- moved R3 0.05 mm to (150.0, 106.6)
- renumbered IC5 to IC1, IC4 to IC2, J4 to J1, J3 to J2, J2 to J3, R4 to R3
Routing:
- net +5V: track 0.00 -> 20.9 mm, vias 0 -> 8
- net Net-(IC3-Y): track 0.00 -> 20.4 mm, vias 0 -> 1
- net LATCH: track 0.00 -> 14.7 mm
- net OMNIPOLAR LATCH: track 0.00 -> 6.58 mm
- net GND: track 0.00 -> 0.37 mm, vias 0 -> 6
- added copper zone on B.Cu, net +5V
- added copper zone on B.Cu, net GND
- added copper zone on F.Cu, net GND
- added copper zone on F.Cu, net Net-(J1-Pin_2)
- added copper zone on B.Cu, net Net-(J3-Pin_1)
- added copper zone on F.Cu, net Net-(J4-Pad1)
Other:
- board size 70 x 9.5 mm -> 70 x 10.5 mm
- board text added: "+"
- board text added: "+5V"
- board text added: "-"
- board text added: "GND"
- board text added: "PT-Main V2.0"
