File: Powered_Torpedo_V2.1/Powered_Torpedo_V2.1.kicad_sch (KiCad schematic)
At the start: 13 parts, among them IC3 AND Gate, IC4 Omnipolar Latch, IC5 Latch, J1 Microfit 3.0, J2 Motor, J3 CAPACITOR #2, J4 CAPACITOR #1, Q1 Mosfet

Commit message: June-1-2025 jlcpcb order
Parts:
- C1, C2: LCSC (none) -> C49678
- IC1: renamed from IC5; value Latch -> A1221: Latch; LCSC (none) -> C2655015
- IC2: renamed from IC4; value Omnipolar Latch -> A3212: Omnipolar Latch; LCSC (none) -> C146383
- IC3: LCSC (none) -> C7434173
- J4: renamed from J1; footprint 0436500302 -> SamacSys_Parts:436500300
- Q1: LCSC (none) -> C145104
- R1, R2: LCSC (none) -> C17414
- renumbered J4 to J1, J3 to J2, J2 to J3, R4 to R3
Changed lines of the file:
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@@
 	(wire
 		(pts
-			(xy 124.46 107.95) (xy 132.08 107.95)
-		)
-		(stroke
-			(width 0)
-			(type default)
-		)
-	)
-	(wire
-		(pts
-			(xy 193.04 144.78) (xy 193.04 151.13)
+			(xy 129.54 107.95) (xy 132.08 107.95)
+		)
+		(stroke
+			(width 0)
+			(type default)
+		)
+	)
+	(wire
+		(pts
+			(xy 193.04 144.78) (xy 193.04 153.67)
 		)
 		(stroke
@@
 	(wire
 		(pts
-			(xy 124.46 105.41) (xy 132.08 105.41)
+			(xy 129.54 105.41) (xy 132.08 105.41)
 		)
 		(stroke
@@
 	(global_label "LATCH"
 		(shape input)
-		(at 124.46 107.95 180)
+		(at 129.54 107.95 180)
 		(fields_autoplaced yes)
 		(effects
@@
 		)
 		(property "Intersheetrefs" "${INTERSHEET_REFS}"
-			(at 115.79 107.95 0)
+			(at 120.87 107.95 0)
 			(effects
 				(font
@@
 	(global_label "LATCH"
 		(shape input)
-		(at 193.04 151.13 180)
+		(at 193.04 153.67 180)
 		(fields_autoplaced yes)
 		(effects
@@
 		)
 		(property "Intersheetrefs" "${INTERSHEET_REFS}"
-			(at 184.37 151.13 0)
+			(at 184.37 153.67 0)
 			(effects
 				(font
@@
 	(global_label "OMNIPOLAR LATCH"
 		(shape input)
-		(at 124.46 105.41 180)
+		(at 129.54 105.41 180)
 		(fields_autoplaced yes)
 		(effects
@@
 		)
 		(property "Intersheetrefs" "${INTERSHEET_REFS}"
-			(at 104.118 105.41 0)
+			(at 109.198 105.41 0)
 			(effects
 				(font
@@
 			)
 		)
+		(property "LCSC" "C17414"
+			(at 116.84 162.56 0)
+			(effects
+				(font
+					(size 1.27 1.27)
+				)
+				(hide yes)
+			)
+		)
 		(pin "1"
 		)
@@
 			)
 		)
+		(property "LCSC" "C7434173"
+			(at 132.08 105.41 0)
+			(effects
+				(font
+					(size 1.27 1.27)
+				)
+				(hide yes)
+			)
+		)
 		(pin "1"
 		)
@@
 			)
 		)
+		(property "LCSC" "C17414"
+			(at 198.12 148.59 0)
+			(effects
+				(font
+					(size 1.27 1.27)
+				)
+				(hide yes)
+			)
+		)
 		(pin "1"
 		)
@@
 				)
 				(justify left top)
+				(hide yes)
+			)
+		)
+		(property "LCSC" "C145104"
+			(at 184.15 105.41 0)
+			(effects
+				(font
+					(size 1.27 1.27)
+				)
 				(hide yes)
 			)
@@
 		(on_board yes)
 		(dnp no)
-		(property "Reference" "J2"
+		(property "Reference" "J3"
 			(at 203.2 83.8201 0)
 			(effects
@@
 			(project "Powered_Torpedo_V2.1"
 				(path "/c3b4e927-b550-45c3-ad51-7ff88d65109a"
-					(reference "J2")
+					(reference "J3")
 					(unit 1)
 				)
@@
 		(on_board yes)
 		(dnp no)
-		(property "Reference" "J1"
+		(property "Reference" "J4"
 			(at 56.896 84.582 0)
 			(effects
@@
 			)
 		)
-		(property "Footprint" "0436500302"
+		(property "Footprint" "SamacSys_Parts:436500300"
 			(at 50.8 183.82 0)
 			(effects
@@
 			(project "Powered_Torpedo_V2.1"
 				(path "/c3b4e927-b550-45c3-ad51-7ff88d65109a"
-					(reference "J1")
+					(reference "J4")
 					(unit 1)
 				)
@@
 		)
 		(property "Description" "Unpolarized capacitor"
+			(at 210.82 146.05 0)
+			(effects
+				(font
+					(size 1.27 1.27)
+				)
+				(hide yes)
+			)
+		)
+		(property "LCSC" "C49678"
 			(at 210.82 146.05 0)
 			(effects
@@
 		(on_board yes)
 		(dnp no)
-		(property "Reference" "J3"
+		(property "Reference" "J2"
 			(at 104.14 113.0299 0)
 			(effects
@@
 			(project "Powered_Torpedo_V2.1"
 				(path "/c3b4e927-b550-45c3-ad51-7ff88d65109a"
-					(reference "J3")
+					(reference "J2")
 					(unit 1)
 				)
@@
 		(dnp no)
 		(fields_autoplaced yes)
-		(property "Reference" "IC4"
+		(property "Reference" "IC2"
 			(at 129.54 134.62 0)
 			(effects
@@
 			)
 		)
-		(property "Value" "Omnipolar Latch"
+		(property "Value" "A3212: Omnipolar Latch"
 			(at 129.54 137.16 0)
 			(effects
@@
 			)
 		)
-		(property "Datasheet" "https://www.allegromicro.com/~/media/files/datasheets/a3211-12-datasheet.pdf"
+		(property "Datasheet" "https://www.allegromicro.com/~/media/Files/Datasheets/A3211-12-Datasheet.ashx"
 			(at 142.24 337.16 0)
 			(effects
@@
 				)
 				(justify left top)
+				(hide yes)
+			)
+		)
+		(property "LCSC" "C146383"
+			(at 113.03 142.24 0)
+			(effects
+				(font
+					(size 1.27 1.27)
+				)
 				(hide yes)
 			)
@@
 			(project "Powered_Torpedo_V2.1"
 				(path "/c3b4e927-b550-45c3-ad51-7ff88d65109a"
-					(reference "IC4")
+					(reference "IC2")
 					(unit 1)
 				)
@@
 		(on_board yes)
 		(dnp no)
-		(property "Reference" "J4"
+		(property "Reference" "J1"
 			(at 104.14 99.0599 0)
 			(effects
@@
 			(project "Powered_Torpedo_V2.1"
 				(path "/c3b4e927-b550-45c3-ad51-7ff88d65109a"
-					(reference "J4")
+					(reference "J1")
 					(unit 1)
 				)
@@
 		(on_board yes)
 		(dnp no)
-		(property "Reference" "R4"
+		(property "Reference" "R3"
 			(at 80.01 109.22 0)
 			(effects
@@
 			(project "Powered_Torpedo_V2.1"
 				(path "/c3b4e927-b550-45c3-ad51-7ff88d65109a"
-					(reference "R4")
+					(reference "R3")
 					(unit 1)
 				)
@@
 		(on_board yes)
 		(dnp no)
-		(property "Reference" "IC5"
+		(property "Reference" "IC1"
 			(at 176.53 152.4 0)
 			(effects
@@
 			)
 		)
-		(property "Value" "Latch"
+		(property "Value" "A1221: Latch"
 			(at 176.53 149.86 0)
 			(effects
@@
 			)
 		)
-		(property "Datasheet" "https://www.allegromicro.com/~/media/files/datasheets/a3211-12-datasheet.pdf"
+		(property "Datasheet" "https://www.allegromicro.com/~/media/Files/Datasheets/A1220-1-2-3-Datasheet.ashx"
 			(at 163.83 337.16 0)
 			(effects
@@
 				)
 				(justify left top)
+				(hide yes)
+			)
+		)
+		(property "LCSC" "C2655015"
+			(at 193.04 142.24 0)
+			(effects
+				(font
+					(size 1.27 1.27)
+				)
 				(hide yes)
 			)
@@
 			(project "Powered_Torpedo_V2.1"
 				(path "/c3b4e927-b550-45c3-ad51-7ff88d65109a"
-					(reference "IC5")
+					(reference "IC1")
 					(unit 1)
 				)
@@
 			(at 95.25 146.05 0)
 			(effects
+				(font
+					(size 1.27 1.27)
+				)
+				(hide yes)
+			)
+		)
+		(property "LCSC" "C49678"
+			(at 95.25 146.05 0)
+			(effects
