File: torpedo_pcbs/Grove_based_board/Grove_based_board.kicad_pcb (KiCad board)
At the start: 4 copper layers, 89 x 31 mm, 91 parts, among them IC10 LIS2MDLTR: Magnetometer, IC2 DRV8213DSGR, IC3 DRV8213DSGR, IC4 DRV8213DSGR, IC5 DRV8213DSGR, IC6 VEML6040A3OG, IC7 AP7362-33SP-13, IC7 AP7362-33SP-13: Batt->3.3V, IC8 TPS76918DBVR, IC8 TPS76918DBVR: 3.3V->1.8V, IC9 TPS60150DRVR: 3.3V->5V, J1 503480-2200, J10 UART Comms, J11 LCD Screen, J12 Conn_01x01, J13 Fan, J2 503480-2200, J3 503480-0440, J4 503480-0440, J5 Push-in Terminals, J6 LiHV (3.8V), J9 MTF-02P Connector, Q1 BSS138, Q2 BSS138, SW1 SW_SPDT, U1 STLINK-V3MINIE Edge Connector, U2 STM32G473CBU6, U3 LSM6DSOTR: Acc+Gyro+Temp, U4 ILPS22QS: Air Pressure+Temp

Commit message: everything is connected
Parts:
- removed C12: 0.1μF, Capacitor_SMD:C_0603_1608Metric
- removed the C22 at (202.1, 94.6)
- removed the C22 at (49.7, 105.6)
- removed the C23 at (202.1, 97.1)
- removed the C23 at (53.7, 90.5)
- removed C28, C29: 22nF, Capacitor_SMD:C_0603_1608Metric
- removed the D1 at (57.7, 90.5)
- removed the D1 at (202.1, 99.6)
- removed F1: Fuse Holder, Capacitor_SMD:C_0603_1608Metric
- removed the IC7 at (47.9, 110.1)
- removed IC8: TPS76918DBVR, SamacSys_Parts:SOT95P280X145-5N
- removed IC8: TPS76918DBVR: 3.3V->1.8V, SamacSys_Parts:SOT95P280X145-5N
- removed J12: Conn_01x01, Connector_PinHeader_1.27mm:PinHeader_1x01_P1.27mm_Vertical
- removed Q1, Q2: BSS138, Package_TO_SOT_SMD:SOT-23
- removed the R6 at (201.4, 105.0)
- removed the R6 at (85.5, 84.6)
- removed SW1: SW_SPDT, Connector_PinSocket_1.27mm:PinSocket_1x02_P1.27mm_Vertical
- added C22: 10μF, Capacitor_SMD:C_0603_1608Metric, F.Cu at (125.9, 81.6)
- added C23: 10μF, Capacitor_SMD:C_0603_1608Metric, F.Cu at (132.3, 86.2)
- added C30: 1μF, Capacitor_SMD:C_0603_1608Metric, F.Cu at (173.0, 85.2)
- added C31: 2.2μF, Capacitor_SMD:C_0603_1608Metric, F.Cu at (176.5, 83.8)
- added C32: 2.2μF, Capacitor_SMD:C_0603_1608Metric, F.Cu at (178.2, 87.2)
- added C33: 0.1μF, Capacitor_SMD:C_0603_1608Metric, F.Cu at (139.8, 92.8)
- added C34: 0.1μF, Capacitor_SMD:C_0603_1608Metric, F.Cu at (140.2, 95.2)
- added C35: 220nF, Capacitor_SMD:C_0603_1608Metric, F.Cu at (144.2, 105.6)
- added D1: LED, Capacitor_SMD:C_0603_1608Metric, F.Cu at (166.4, 109.7)
- added F2: Fuse Holder, SamacSys_Parts:0154001.DRT, F.Cu at (111.6, 82.5)
- added H4: MountingHole, MountingHole:MountingHole_2.2mm_M2, F.Cu at (136.5, 108.4)
- added J7: Batt-, Connector_PinHeader_2.54mm:PinHeader_1x01_P2.54mm_Vertical, F.Cu at (103.6, 108.9)
- added J8: MTF-02P Connector, Connector_PinSocket_1.27mm:PinSocket_1x04_P1.27mm_Vertical, F.Cu at (177.3, 81.9)
- added Q5: DMG1013UW-7, SamacSys_Parts:2SC2712GRLF, F.Cu at (163.9, 83.0)
- added Q6: PMOS SI4435FDY, SamacSys_Parts:SOIC127P600X175-8N, F.Cu at (121.2, 82.8)
- added Q7: NMOS, SamacSys_Parts:SOTFL95P240X88-3N, F.Cu at (121.0, 90.2)
- added R22: 10k, Resistor_SMD:R_0603_1608Metric, F.Cu at (114.7, 88.7)
- added R23: 100k, Resistor_SMD:R_0603_1608Metric, F.Cu at (115.7, 90.1)
- added R6: 350, Resistor_SMD:R_0603_1608Metric, F.Cu at (169.7, 109.7)
- added S1: MSK12C02, SamacSys_Parts:MSK12C02, F.Cu at (118.2, 108.5)
- added SW2: SW_SPST, SamacSys_Parts:436331045822, B.Cu at (161.5, 81.7)
- added SW3: SW_SPST, SamacSys_Parts:436331045822, B.Cu at (169.0, 81.7)
- added SW4: SW_SPST, SamacSys_Parts:436331045822, B.Cu at (154.0, 81.7)
- added SW5: button, SamacSys_Parts:B3U3100PMB, F.Cu at (101.0, 81.8)
- added Y2: 16MHz, SamacSys_Parts:X322516MOB4SI, F.Cu at (123.8, 88.2)
- A2: footprint board_board_connection:Grove conn -> board_board_connection:Grove conn_limited_pinout
- C10: value 1μF -> 0.1μF
- C11: value 2.2μF -> 0.1μF
- C24, C26: value ??μF -> 12μF
- C5: value 0.1μF -> 1μF
- C7, IC10, J1, J2: moved to F.Cu
- D2, D3, D4: footprint Capacitor_SMD:C_0603_1608Metric -> LED_SMD:LED_0805_2012Metric
- H3: value 22pin->15pin Adapter Slot -> MountingHole; footprint MountingEquipment:slot -> MountingHole:MountingHole_2.2mm_M2
- J10, J11: footprint Connector_PinSocket_2.00mm:PinSocket_2x02_P2.00mm_Vertical -> SamacSys_Parts:BM04B-SRSS-TB_LFSN_
- J13: value Fan -> I2C2 Access; footprint Connector_PinSocket_1.27mm:PinSocket_1x02_P1.27mm_Vertical -> SamacSys_Parts:BM04B-SRSS-TB_LFSN_
- J6: value LiHV (3.8V) -> Batt+; footprint Connector_PinHeader_2.54mm:PinHeader_1x02_P2.54mm_Vertical -> Connector_PinHeader_2.54mm:PinHeader_1x01_P2.54mm_Vertical
- J9: value MTF-02P Connector -> I2C2 Access; footprint Connector_PinSocket_2.00mm:PinSocket_2x02_P2.00mm_Vertical -> SamacSys_Parts:BM04B-SRSS-TB_LFSN_
- R10: value R -> 260; footprint Resistor_SMD:R_0201_0603Metric -> Resistor_SMD:R_0603_1608Metric
- R11, R9: value R -> 100; footprint Resistor_SMD:R_0201_0603Metric -> Resistor_SMD:R_0603_1608Metric
- R12, R13, R14, R15, R16, R17, R5, R7, R8: footprint Resistor_SMD:R_0201_0603Metric -> Resistor_SMD:R_0603_1608Metric
- R18: value ??? -> 1.5k; footprint Resistor_SMD:R_0201_0603Metric -> Resistor_SMD:R_0603_1608Metric
- moved D3 121.4 mm to (178.4, 108.7), turned to 90 degrees
- moved D4 119.1 mm to (176.3, 108.7), turned to 90 degrees
- moved D2 117.6 mm to (174.3, 108.7), turned to 90 degrees
- moved C11 97.2 mm to (142.2, 106.7), turned to 90 degrees
- moved R10 93.2 mm to (178.4, 105.4), turned to -90 degrees
- moved R11 90.8 mm to (176.3, 105.4), turned to -90 degrees
- moved R9 90.1 mm to (174.3, 105.4), turned to -90 degrees
- moved C27 88.4 mm to (141.7, 109.5)
- moved C13 85.8 mm to (130.3, 87.0), turned to 135 degrees
- moved C15 85.4 mm to (129.2, 88.0), turned to 135 degrees
- moved C17 84.4 mm to (134.0, 96.2), turned to 45 degrees
- moved J10 81.1 mm to (157.7, 109.0)
- moved C14 79.6 mm to (125.3, 101.0), turned to 180 degrees
- moved C16 78.6 mm to (128.2, 89.1), turned to -45 degrees
- moved R12 78.1 mm to (166.1, 86.4), turned to 90 degrees
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Connections:
- net FAN renamed STM32_PC13
- net Net-(IC10-SCL/SPC) renamed /SCL_MAG
- net Net-(IC10-SDA/SDI/SDO) renamed /SDA_MAG
- A1 pad 10: MODE_SEL_DIAL1 -> MODE_SEL_UP
- A1 pad 11: MODE_SEL_SWITCH -> MODE_SEL_ENTER
- A1 pad 12: +3.3V -> /ESP32_3.3V
- A1 pad 14: unconnected-(A1-BAT--Pad14) -> /ESP32_pmos_gate
- A1 pad 9: MODE_SEL_DIAL2 -> MODE_SEL_DOWN
- C10 pad 1: +3.3V -> POWER_SHUTOFF
- C11 pad 1: +1V8 -> +3.3V
- C26 pad 2: Net-(C26-Pad2) -> /HSE_OUT
- C5 pad 1: Net-(IC1-REGOUT) -> /PMOS_drain
- C5 pad 2: GND -> +BATT
- IC2 pad 5: MOTOR0_IN -> MOTOR0_PWM
- IC2 pad 6: MOTOR0_PWM -> MOTOR0_IN
- IC3 pad 5: MOTOR1_IN -> MOTOR1_PWM
- IC3 pad 6: MOTOR1_PWM -> MOTOR1_IN
- IC4 pad 5: MOTOR2_IN -> MOTOR2_PWM
- IC4 pad 6: MOTOR2_PWM -> MOTOR2_IN
- IC5 pad 5: MOTOR3_IN -> MOTOR3_PWM
- IC5 pad 6: MOTOR3_PWM -> MOTOR3_IN
- IC7 pad 5: Net-(IC7-OUT_1) -> +3.3V
- IC7 pad 7: unconnected-(IC7-OUT_3-Pad7) -> +3.3V
- J10 pad 1: +3.3V -> unconnected-(J10-Pin_1-Pad1)
- J10 pad 2: Net-(A1-D7/RX/SS) -> Net-(A1-D6/TX)
- J10 pad 3: Net-(A1-D6/TX) -> Net-(A1-D7/RX/SS)
- J13 pad 1: +3.3V -> STM32_PB2
- J13 pad 2: Net-(J13-Pin_2) -> STM32_PB5
- J4 pad 3: LIGHT -> unconnected-(J4-Pad3)
- J6 pad 1: Net-(J6-Pin_1) -> /Batt_terminal+
- J9 pad 1: +5V -> +3.3V
- J9 pad 2: OPT_FLOW_RX -> SCL2
- J9 pad 3: OPT_FLOW_TX -> SDA2
- R12 pad 1: Net-(S1-ChannelB) -> GND
- R12 pad 2: MODE_SEL_DIAL2 -> /ESP32_pmos_gate
- R15 pad 1: +3.3V -> MODE_SEL_ENTER
- R15 pad 2: Net-(S1-ChannelA) -> GND
- R16 pad 1: +3.3V -> MODE_SEL_UP
- R16 pad 2: Net-(S1-ChannelB) -> GND
- R17 pad 1: Net-(S1-ChannelA) -> MODE_SEL_DOWN
- R17 pad 2: MODE_SEL_DIAL1 -> GND
- R18 pad 1: /HSE_OUT -> /PMOS_drain
- R18 pad 2: Net-(C26-Pad2) -> /NMOS_drain
- U2 pad 10: MOTOR0_PWM -> MOTOR0_IN
- U2 pad 11: MOTOR0_IN -> MOTOR0_PWM
- U2 pad 18: MOTOR2_PWM -> MOTOR2_IN
- U2 pad 19: /UNUSED ADC -> STM32_PB2
- U2 pad 22: MOTOR2_IN -> MOTOR2_PWM
- U2 pad 33: LIGHT_COMMS -> STM32_PA11
- U2 pad 4: INV_POWER_SHUTOFF -> POWER_SHUTOFF
- U2 pad 43: unconnected-(U2-PB5-Pad43) -> STM32_PB5
- U2 pad 44: OPT_FLOW_TX -> unconnected-(U2-PB6-Pad44)
Routing:
- net GND: track 0.00 -> 101.2 mm, vias 0 -> 42
- net +3.3V: track 0.00 -> 79.3 mm, vias 0 -> 19
- net SDA4: track 0.00 -> 62.2 mm, vias 0 -> 3
- net STM32_DEBUG_LED1: track 0.00 -> 61.0 mm, vias 0 -> 2
- net GROVE_DEBUG_LED1: track 0.00 -> 60.8 mm, vias 0 -> 1
- net OPT_FLOW_RX: track 0.00 -> 59.7 mm
- net SCL4: track 0.00 -> 44.2 mm, vias 0 -> 5
- net SDA2: track 0.00 -> 44.0 mm, vias 0 -> 2
- net ESP32_DEBUG_LED1: track 0.00 -> 42.3 mm, vias 0 -> 2
- net SCL2: track 0.00 -> 41.2 mm, vias 0 -> 2
- net GROVE_RST: track 0.00 -> 41.1 mm, vias 0 -> 1
- net MODE_SEL_DOWN: track 0.00 -> 31.2 mm, vias 0 -> 1
- net STM32_NRST: track 0.00 -> 29.5 mm, vias 0 -> 2
- net MODE_SEL_UP: track 0.00 -> 26.8 mm, vias 0 -> 1
- net /NMOS_drain: track 0.00 -> 26.5 mm, vias 0 -> 2
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- added copper zone on B.Cu, net +3.3V
- added copper zone on F.Cu, net +3.3V
- added copper zone on F.Cu, net +3.3VA
- added copper zone on F.Cu, net +5V
- added copper zone on B.Cu, net +BATT
- added copper zone on F.Cu, net +BATT
- added copper zone on F.Cu, net /Batt_terminal+
- added copper zone on F.Cu, net /Motor driver0/OUT1
- added copper zone on F.Cu, net /Motor driver0/OUT2
- added copper zone on F.Cu, net /Motor driver1/OUT1
- added copper zone on F.Cu, net /Motor driver1/OUT2
- added copper zone on F.Cu, net /Motor driver2/OUT1
- added copper zone on F.Cu, net /Motor driver2/OUT2
- added copper zone on F.Cu, net /Motor driver3/OUT1
- added copper zone on F.Cu, net /Motor driver3/OUT2
- added copper zone on F.Cu, net /PMOS_drain
- added copper zone on B.Cu, net GND
- added copper zone on F.Cu, net GND
Other:
- board size 89 x 31 mm -> 88.6 x 31 mm

Commit message: June-1-2025 jlcpcb order
Parts:
- removed C35: 220nF, Capacitor_SMD:C_0603_1608Metric
- removed IC10: LIS2MDLTR: Magnetometer, SamacSys_Parts:LGA-12
- removed Q5: DMG1013UW-7, SamacSys_Parts:2SC2712GRLF
- removed S1: MSK12C02, SamacSys_Parts:MSK12C02
- removed U3: LSM6DSOTR: Acc+Gyro+Temp, SamacSys_Parts:LGA-14L_2P5X3X0P86_STM
- added C12: 10μF, Capacitor_SMD:C_0603_1608Metric, F.Cu at (144.3, 105.5)
- added C28: 1μF, Capacitor_SMD:C_0603_1608Metric, F.Cu at (149.2, 109.2)
- added C29: 0.1μF, Capacitor_SMD:C_0603_1608Metric, F.Cu at (141.6, 94.3)
- added G***: LOGO, LOGO, B.Cu at (141.6, 108.2)
- added IC1: ICM-42688-P, SamacSys_Parts:IIM42352, F.Cu at (139.4, 95.5)
- added IC8: MMC5983MA-B, SamacSys_Parts:MMC5983MAB, F.Cu at (146.6, 108.5)
- added J14: LCD Screen, SamacSys_Parts:BM04B-SRSS-TB_LFSN_, F.Cu at (153.1, 108.0)
- added Q1: SI1967DH-T1-GE3, SamacSys_Parts:SOT65P210X110-6N, F.Cu at (164.5, 84.6)
- added R19: 10k, Resistor_SMD:R_0603_1608Metric, F.Cu at (124.0, 99.2)
- added SW1: button, SamacSys_Parts:B3U3100PMB, F.Cu at (115.2, 108.6)
- added TH1: 10k, Resistor_SMD:R_1206_3216Metric, B.Cu at (131.5, 99.3)
- C24, C26: value 12μF -> 12pF
- C30: value 1μF -> 2.2μF
- C33: value 0.1μF -> 2.2μF
- C34: value 0.1μF -> 10nF
- D1: footprint Capacitor_SMD:C_0603_1608Metric -> LED_SMD:LED_0805_2012Metric
- FB1: value FerriteBead -> 120R
- J1, J2: value 503480-2200 -> FH34SRJ-22S-0.5SH_99_; footprint SamacSys_Parts:5034802200 -> SamacSys_Parts:FH34SRJ22S05SH99
- J10: value UART Comms -> 1770940; footprint SamacSys_Parts:BM04B-SRSS-TB_LFSN_ -> SamacSys_Parts:1770940
- J11: value LCD Screen -> I2C2 Access
- J13: value I2C2 Access -> GPIO Access; footprint SamacSys_Parts:BM04B-SRSS-TB_LFSN_ -> Connector_PinHeader_1.27mm:PinHeader_1x04_P1.27mm_Vertical
- J3, J4: value 503480-0440 -> FH34SRJ-4S-0.5SH_50_; footprint SamacSys_Parts:5034800440 -> SamacSys_Parts:FH34SRJ4S05SH50
- J5: value Push-in Terminals -> Conn_01x01; footprint SamacSys_Parts:009276008021106 -> Connector_PinHeader_1.00mm:PinHeader_1x01_P1.00mm_Vertical
- J9: value I2C2 Access -> LCD Screen
- Q6: value PMOS SI4435FDY -> PMOS
- R1, R2, R3, R4: footprint Resistor_SMD:R_0805_2012Metric -> Resistor_SMD:R_0603_1608Metric
- R10: value 260 -> 200
- R11, R9: value 100 -> 200
- R5: value 10k -> 1.5k
- R6: value 350 -> 200
- U2: value STM32G473CBU6 -> STM32G431CBUx
- moved J10 59.5 mm to (99.8, 95.5), turned to -90 degrees
- moved J5 49.0 mm to (148.6, 106.1), turned to 0 degrees
- moved J9 32.3 mm to (160.4, 108.0)
- moved R5 23.4 mm to (143.6, 92.4), turned to -90 degrees
- moved J11 18.9 mm to (130.9, 107.7)
- moved J13 4.78 mm to (111.4, 109.6), turned to -90 degrees
- moved R7 3.20 mm to (133.5, 104.7), turned to 180 degrees
- moved R8 3.10 mm to (130.3, 104.8), turned to 0 degrees
- moved J1 2.93 mm to (173.6, 95.5), turned to 90 degrees
- moved J2 2.92 mm to (168.9, 95.5), turned to -90 degrees
- moved C27 2.67 mm to (140.1, 107.4), turned to 120 degrees
- moved C34 2.60 mm to (141.2, 97.7), turned to -105 degrees
- moved IC6 1.72 mm to (140.9, 109.5), turned to 0 degrees
- moved R22 1.57 mm to (115.8, 89.8)
- moved U4 1.56 mm to (142.8, 109.0), turned to 90 degrees
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Connections:
- net /ESP32_pmos_gate renamed /ESP32PowGate
- net /PMOS_drain renamed /PMOS_source
- C21 pad 2: STM32_NRST -> Net-(SW1-B)
- J10 pad 1: unconnected-(J10-Pin_1-Pad1) -> /Motor driver0/OUT1
- J10 pad 2: Net-(A1-D6/TX) -> /Motor driver0/OUT1
- J10 pad 3: Net-(A1-D7/RX/SS) -> /Motor driver0/OUT2
- J10 pad 4: GND -> /Motor driver0/OUT2
- J10 pad 5: (no net) -> /Motor driver1/OUT1
- J10 pad 6: (no net) -> /Motor driver1/OUT1
- J11 pad 2: SCL4 -> SCL2
- J11 pad 3: SDA4 -> SDA2
- J11 pad 5: (no net) -> GND
- J11 pad 6: (no net) -> GND
- J13 pad 1: STM32_PB2 -> unconnected-(J13-Pin_1-Pad1)
- J13 pad 3: STM32_PA11 -> STM32_PC13
- J13 pad 4: STM32_PA11 -> STM32_PC14
- J3 pad 2: +3.3V -> SDA2
- J3 pad 3: SDA2 -> +3.3V
- J4 pad 1: GPIO1 -> +3.3V
- J4 pad 2: XSHUT -> GND
- J4 pad 3: unconnected-(J4-Pad3) -> GPIO1
- J4 pad 4: unconnected-(J4-Pad4) -> XSHUT
- J5 pad 1: /Motor driver0/OUT1 -> Net-(IC8-INT)
- J9 pad 1: +3.3V -> unconnected-(J9-Pin_1-Pad1)
- J9 pad 2: SCL2 -> Net-(A1-D6/TX)
- J9 pad 3: SDA2 -> Net-(A1-D7/RX/SS)
- J9 pad 5: (no net) -> GND
- J9 pad 6: (no net) -> GND
- R5 pad 1: /BOOT0_STM -> STM32_NRST
- R5 pad 2: Net-(S1-COM) -> Net-(SW1-B)
- R7 pad 2: SCL2 -> SDA2
- R8 pad 2: SDA2 -> SCL2
- U1 pad 8: TX -> RX_STLINK
- U1 pad 9: RX -> TX_STLINK
- U2 pad 19: STM32_PB2 -> /Batt_temp
- U2 pad 29: SCL4 -> IMU_int
- U2 pad 3: BATT_TEMP -> STM32_PC14
- U2 pad 30: SCL2 -> SDA2
- U2 pad 31: SDA2 -> SCL2
- U2 pad 33: STM32_PA11 -> GPIO1
- U2 pad 34: IMU_INT -> XSHUT
- U2 pad 39: TX -> TX_STLINK
- U2 pad 40: RX -> RX_STLINK
- U2 pad 46: /BOOT0_STM -> SCL4
- U2 pad 7: STM32_NRST -> Net-(SW1-B)
Routing:
- net Net-(SW1-B): track 0.00 -> 64.3 mm, vias 0 -> 2
- net XSHUT: track 2.12 -> 44.9 mm, vias 0 -> 2
- net SCL2: track 41.2 -> 82.1 mm, vias 2 -> 4
- net GPIO1: track 2.58 -> 43.4 mm, vias 0 -> 2
- net STM32_PC14: track 0.00 -> 37.3 mm, vias 0 -> 1
- net STM32_PC13: track 0.00 -> 36.2 mm, vias 0 -> 1
- net SDA2: track 44.0 -> 80.1 mm, vias 2 -> 8
- net STM32_PB5: track 0.00 -> 35.0 mm, vias 0 -> 1
- net STM32_NRST: track 29.5 -> 3.31 mm, vias 2 -> 0
- net /BOOT0_STM: track 21.7 -> 0.00 mm, vias 2 -> 0
- net +3.3V: track 79.3 -> 99.2 mm, vias 19 -> 22
- net TX_STLINK: track 0.00 -> 19.6 mm, vias 0 -> 1
- net RX: track 18.5 -> 0.00 mm, vias 1 -> 0
- net RX_STLINK: track 0.00 -> 18.3 mm, vias 0 -> 1
- net TX: track 16.2 -> 0.00 mm, vias 1 -> 0
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- added copper zone on In1.Cu, net +BATT
- added copper zone on In1.Cu, net /Batt_terminal+
- added copper zone on In2.Cu, net /Batt_terminal+
- added copper zone on In1.Cu, net /PMOS_source
Other:
- board text added: "---"
- board text added: "1"
- board text added: "2"
- board text added: "A"
- board text added: "AT-Main V1"
- board text added: "Batt+"
- board text added: "Batt-"
- board text added: "C"
- board text added: "ESP"
- board text added: "G"
- board text added: "Grove"
- board text added: "PB5"
- board text added: "PC13"
- board text added: "PC14"
- board text added: "R"
- board text added: "STM"
- board text added: "T"
- board text added: "V"
- board text added: "[Battery goes here]"
