File: torpedo_pcbs/Grove_based_board/Grove_based_board.kicad_sch (KiCad schematic)
At the start: 2 parts

Commit message: sensors pcb and main pcb improvements
Parts:
- removed A2: Grove AI Vision Module V2, board_board_connection:Grove_ai_vision_module_v2_headerless, symbol board-connections:Grove-AI-Vision-Module-V2
- added H1, H2: MountingHole, MountingHole:MountingHole_2.2mm_M2, symbol Mechanical:MountingHole
- added IC1: ICM-20948, QFN40P300X300X105-25N-D, symbol SamacSys_Parts:ICM-20948
- added IC6: STM32G473CBU6, QFN50P700X700X60-49N-D, symbol SamacSys_Parts:STM32G473CBU6
- added IC7: AP7362-33SP-13, SOIC127P600X150-9N, symbol SamacSys_Parts:AP7362-33SP-13
- added J1, J2: 503480-2200, 5034802200, symbol SamacSys_Parts:503480-2200
- added J3, J4: 503480-0440, 5034800440, symbol SamacSys_Parts:503480-0440
- added J5: S8B-EH, SHDRRA8W64P0X250_1X8_2250X820X420P, symbol SamacSys_Parts:S8B-EH
- added J6: Conn_01x02, Connector_PinHeader_2.54mm:PinHeader_1x02_P2.54mm_Vertical, symbol Connector_Generic:Conn_01x02
Connections:
- net GND: now also IC7.1 (GND), IC7.9 (EP), J1.MP1, J1.MP2, J2.MP1, J2.MP2, J3.4, J3.MP1, J3.MP2, J4.MP1, J4.MP2, J6.2 (Pin_2)
- net SCL: now also J3.1
- net SDA: now also J3.3
- new net: J1.1, J2.22
- new net: J1.10, J2.13
- new net: J1.11, J2.12
- new net: J1.12, J2.11
- new net: J1.13, J2.10
- new net: J1.14, J2.9
- new net: J1.15, J2.8
- new net: J1.16, J2.7
- new net: J1.17, J2.6
- new net: J1.18, J2.5
- new net: J1.19, J2.4
- new net: J1.2, J2.21
- new net: J1.20, J2.3
- new net: J1.21, J2.2
- new net: J1.22, J2.1
- new net: J1.3, J2.20
- new net: J1.4, J2.19
- new net: J1.5, J2.18
- new net: J1.6, J2.17
- new net: J1.7, J2.16
- new net: J1.8, J2.15
- new net: J1.9, J2.14
- new net +3.3V: IC7.5 (OUT_1), IC7.6 (OUT_2), IC7.7 (OUT_3), J3.2
- new net +BATT: IC7.2 (EN), IC7.3 (IN_1), IC7.4 (IN_2), J6.1 (Pin_1)
- new net GPIO1: J4.1
- new net LIGHT: J4.3
- new net Motor driver0/OUT1: J5.1
- new net Motor driver0/OUT2: J5.2
- new net Motor driver1/OUT1: J5.3
- new net Motor driver1/OUT2: J5.4
- new net Motor driver2/OUT1: J5.5
- new net Motor driver2/OUT2: J5.6
- new net Motor driver3/OUT1: J5.7
- new net Motor driver3/OUT2: J5.8
- new net XSHUT: J4.2
- no-connect marks 7 -> 12
Other:
- added sheet Motor driver0 (motor_driver.kicad_sch)
- added sheet Motor driver1 (motor_driver.kicad_sch)
- added sheet Motor driver2 (motor_driver.kicad_sch)
- added sheet Motor driver3 (motor_driver.kicad_sch)
- note added: "Flex connectors"
- note added: "Power"
- moved on the sheet: A1

Commit message: save feb21
Parts:
- removed IC6: STM32G473CBU6, QFN50P700X700X60-49N-D, symbol SamacSys_Parts:STM32G473CBU6
- added C10, C18, C20, C25: 1μF, Capacitor_SMD:C_0603_1608Metric, symbol Device:C
- added C11: 2.2μF, Capacitor_SMD:C_0603_1608Metric, symbol Device:C
- added C12, C14, C15, C16, C17, C21, C27, C5: 0.1μF, Capacitor_SMD:C_0603_1608Metric, symbol Device:C
- added C13, C22, C23: 10μF, Capacitor_SMD:C_0603_1608Metric, symbol Device:C
- added C19: 10nF, Capacitor_SMD:C_0603_1608Metric, symbol Device:C
- added C24, C26: ??μF, Capacitor_SMD:C_0603_1608Metric, symbol Device:C
- added C28, C29: 22nF, Capacitor_SMD:C_0603_1608Metric, symbol Device:C
- added D1, D2, D3, D4: LED, Capacitor_SMD:C_0603_1608Metric, symbol Device:LED
- added F1: Fuse, Capacitor_SMD:C_0603_1608Metric, symbol Device:Fuse
- added FB1: FerriteBead, Capacitor_SMD:C_0603_1608Metric, symbol Device:FerriteBead
- added IC6: VEML6040A3OG, SamacSys_Parts:VEML6040A3OG, symbol SamacSys_Parts:VEML6040A3OG
- added IC8: TPS76918DBVR, SamacSys_Parts:SOT95P280X145-5N, symbol SamacSys_Parts:TPS76918DBVR
- added J10: UART Comms, Connector_PinSocket_2.00mm:PinSocket_2x02_P2.00mm_Vertical, symbol Connector_Generic:Conn_01x04
- added J11: LCD Screen, Connector_PinSocket_2.00mm:PinSocket_2x02_P2.00mm_Vertical, symbol Connector_Generic:Conn_01x04
- added J12: Conn_01x01, Connector_PinHeader_1.27mm:PinHeader_1x01_P1.27mm_Vertical, symbol Connector_Generic:Conn_01x01
- added J13: Fan, Connector_PinSocket_1.27mm:PinSocket_1x02_P1.27mm_Vertical, symbol Connector_Generic:Conn_01x02
- added J7, J8: Conn_01x07, Connector_PinHeader_2.54mm:PinHeader_1x07_P2.54mm_Vertical, symbol Connector_Generic:Conn_01x07
- added J9: UPIXEL Connector, Connector_PinSocket_2.00mm:PinSocket_2x02_P2.00mm_Vertical, symbol Connector_Generic:Conn_01x04
- added Q1, Q2: BSS138, Package_TO_SOT_SMD:SOT-23, symbol Transistor_FET:BSS138
- added Q3: NMOS, symbol Simulation_SPICE:NMOS
- added R10, R11, R6, R9: R, Resistor_SMD:R_0201_0603Metric, symbol Device:R
- added R12, R14, R15, R16, R17, R5: 10k, Resistor_SMD:R_0201_0603Metric, symbol Device:R
- added R13: 20k, Resistor_SMD:R_0201_0603Metric, symbol Device:R
- added R18: ???, Resistor_SMD:R_0201_0603Metric, symbol Device:R
- added R7, R8: 2.2k, Resistor_SMD:R_0201_0603Metric, symbol Device:R
- added S1: Scroll wheel encoder, switches_and_dials:EN10HT1212N5HH3, symbol switches dials and such:EN10HT1212N5HH3
- added SW1: SW_SPDT, Connector_PinSocket_1.27mm:PinSocket_1x02_P1.27mm_Vertical, symbol Switch:SW_SPDT
- added U1: STLINK-V3MINIE Edge Connector, edge connector:STLINK-V3MINIE conn, symbol stm_debug_conn:STLINK-V3MINIE_Connector
- added U2: STM32G473CBU6, Package_DFN_QFN:QFN-48-1EP_7x7mm_P0.5mm_EP5.6x5.6mm, symbol MCU_ST_STM32G4:STM32G473CBUx
- added Y2: 32MHz?, symbol Device:Crystal_GND24
- IC1: footprint QFN40P300X300X105-25N-D -> SamacSys_Parts:QFN40P300X300X105-25N-D
- IC7: footprint SOIC127P600X150-9N -> SamacSys_Parts:SOIC127P600X150-9N
- J1, J2: footprint 5034802200 -> SamacSys_Parts:5034802200
- J3, J4: footprint 5034800440 -> SamacSys_Parts:5034800440
- J5: value S8B-EH -> Push-in Terminals; footprint SHDRRA8W64P0X250_1X8_2250X820X420P -> SamacSys_Parts:motor wire conn; Arrow Part Number (none) -> 009276008021106; Arrow Price/Stock (none) -> https://www.arrow.com/en/products/009276008021106/avx; Height 4.2 -> 5; Manufacturer_Name JST (JAPAN SOLDERLESS TERMINALS) -> Kyocera AVX; Manufacturer_Part_Number S8B-EH -> 009276008021106; Mouser Part Number (none) -> 581-009276008021106; Mouser Price/Stock (none) -> https://www.mouser.co.uk/ProductDetail/AVX/009276008021106?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
- J6: value Conn_01x02 -> LiHV (3.8V)
Connections:
- net +3.3V: now also A1.12 (3V3), IC1.13 (VDD), IC1.22 (NCS), C10.1, C13.1, C14.1, C15.1, C16.2, C17.1, C20.2, C23.1, C27.1, D1.2 (A), FB1.1, IC6.4 (VDD), IC8.1 (IN), J10.1 (Pin_1), J11.1 (Pin_1), J13.1 (Pin_1), J8.3 (Pin_3), Q1.1 (G), Q2.1 (G), R15.1, R16.1, R7.1, R8.1, SW1.1 (A), U1.6 (VCC), U2.1 (VBAT), U2.23 (VDD), U2.35 (VDD), U2.48 (VDD)
- net +BATT: now also C22.1, F1.2, J9.1 (Pin_1), R13.2; no longer J6.1 (Pin_1)
- net GND: now also A1.13 (GND), IC1.11 (FSYNC), IC1.18 (GND), IC1.20 (RESV_2), IC1.9 (SDO_/_AD0), C10.2, C11.2, C12.2, C13.2, C14.2, C15.2, C16.1, C17.2, C18.1, C19.2, C20.1, C21.1, C22.2, C23.2, C24.1, C25.2, C26.1, C27.2, C28.2, C29.2, C5.2, D2.1 (K), D3.1 (K), D4.1 (K), IC6.1 (GND), IC8.2 (GND), IC8.3 (~{EN}), J10.4 (Pin_4), J11.4 (Pin_4), J8.2 (Pin_2), J9.4 (Pin_4), Q3.3 (S), R14.1, R6.2, S1.1 (Common), S1.4 (MH_1), S1.5 (MH_2), SW1.3 (C), U1.10 (GND), U2.49 (VSS), Y2.2, Y2.4; no longer A1.19 (GND), A1.25 (GND)
- net at IC1.10 (REGOUT): now also C5.1
- net IMU_INT: now reaches IC1.12 (INT1)
- net IMU_INT: now also U2.34 (PA12)
- net SCL2: now reaches IC1.23 (SCL_/_SCLK)
- net SCL2: now also J3.1, IC6.3 (SCL), R7.2, U2.30 (PA8)
- net SDA2: now reaches IC1.24 (SDA_/_SDI)
- net SDA2: now also J3.3, IC6.2 (SDA), R8.2, U2.31 (PA9)
- net +1V8: now reaches IC1.8 (VDDIO)
- net +1V8: now also C11.1, C12.1, IC8.5 (OUT)
- net GROVE_RST: now reaches A1.1 (D0/A0)
- net GROVE_RST: now also J7.4 (Pin_4)
- net MODE_SEL_DIAL1: now reaches A1.10 (D9/A9/MISO)
- net MODE_SEL_DIAL1: now also R17.2
- net MODE_SEL_SWITCH: now reaches A1.11 (D10/A10/MOSI)
- net STM32_NRST: now reaches A1.2 (D1/A1)
- net STM32_NRST: now also C21.2, U2.7 (PG10)
- net ESP32_DEBUG_LED1: now reaches A1.3 (D2/A2)
- net ESP32_DEBUG_LED1: now also R10.1
- net at A1.7 (D6/TX): now also J10.3 (Pin_3)
- net at A1.8 (D7/RX/SS): now also J10.2 (Pin_2)
- net MODE_SEL_DIAL2: now reaches A1.9 (D8/A8/SCK)
- net MODE_SEL_DIAL2: now also R12.2
- net SCL renamed SCL4
- net SCL4: now also J11.2 (Pin_2), J7.6 (Pin_6), U2.29 (PC6); no longer J3.1
- net SDA renamed SDA4
- net SDA4: now also J11.3 (Pin_3), J7.5 (Pin_5), U2.45 (PB7); no longer J3.3
- new net: D4.2 (A), R11.2
- new net: R5.2, SW1.2 (B)
- new net: C29.1, R15.2, R17.1, S1.2 (ChannelA)
- new net: C28.1, R12.1, R16.2, S1.3 (ChannelB)
- new net: C26.2, R18.2, Y2.3
- new net: F1.1, J6.1 (Pin_1)
- new net: D3.2 (A), R10.2
- new net: D2.2 (A), R9.2
- new net: D1.1 (K), R6.1
- new net: J13.2 (Pin_2), Q3.1 (D)
- new net +3.3VA: C18.2, C19.1, C25.1, FB1.2, U2.20 (VREF+), U2.21 (VDDA)
- new net BATT_ADC: R13.1, R14.2, U2.24 (PB11)
- new net BATT_TEMP: U2.3 (PC14)
- new net BOOT0_STM: R5.1, U2.46 (PB8)
- new net FAN: Q3.2 (G), U2.2 (PC13)
- new net GROVE_DEBUG_LED1: J7.3 (Pin_3), R9.1
- new net HSE_IN: C24.2, U2.5 (PF0), Y2.1
- new net HSE_OUT: R18.1, U2.6 (PF1)
- new net INV_POWER_SHUTOFF: U2.4 (PC15)
- new net JTCK: U1.2 (CLK), U2.37 (PA14)
- new net JTDI: U1.4 (TDI), U2.38 (PA15)
- new net JTDO: U1.1 (TDO), U2.41 (PB3)
- new net JTMS: U1.3 (TMS), U2.36 (PA13)
- new net JTRST: U1.7 (RST), U2.42 (PB4)
- new net LIGHT_COMMS: U2.33 (PA11)
- new net MOTOR0_GAINSEL: U2.9 (PA1)
- new net MOTOR0_IN: U2.11 (PA3)
- new net MOTOR0_IPROPI: U2.8 (PA0)
- new net MOTOR0_PWM: U2.10 (PA2)
- new net MOTOR1_GAINSEL: U2.14 (PA6)
- new net MOTOR1_IN: U2.15 (PA7)
- new net MOTOR1_IPROPI: U2.12 (PA4)
- new net MOTOR1_PWM: U2.13 (PA5)
- new net MOTOR2_GAINSEL: U2.17 (PB0)
- new net MOTOR2_IN: U2.22 (PB10)
- new net MOTOR2_IPROPI: U2.16 (PC4)
- new net MOTOR2_PWM: U2.18 (PB1)
- new net MOTOR3_GAINSEL: U2.26 (PB13)
- new net MOTOR3_IN: U2.25 (PB12)
- new net MOTOR3_IPROPI: U2.28 (PB15)
- new net MOTOR3_PWM: U2.27 (PB14)
- new net OPT_FLOW_RX: J9.2 (Pin_2), Q1.3 (D), Q2.2 (S), U2.32 (PA10)
- new net OPT_FLOW_TX: J9.3 (Pin_3), Q1.2 (S), Q2.3 (D), U2.44 (PB6)
- new net RX: U1.9 (RX), U2.40 (PC11)
- new net STM32_DEBUG_LED1: R11.1, U2.47 (PB9)
- new net TX: U1.8 (TX), U2.39 (PC10)
- new net UNUSED ADC: J12.1 (Pin_1), U2.19 (PB2)
- no-connect marks 12 -> 40
Other:
- note added: "0.2-2Ω ESR!!!"
- note added: "Grove AI Module V2 Connection"
- note added: "Microcontroller Assemblies"
- note added: "Misc"
- note added: "Motor Controllers"
- note added: "Place close to each VDD pin"
- note added: "SDA4/SCL4 are already pulled up by the Grove AI Vision Module V2 (with 2.2kΩ)"
- note added: "STM32G4 Setup"
- note added: "Sensors / I2C Devices"
- note added: "Setup taken from: https://youtu.be/aVUqaB0IMh4?si=XPnxRO8Demq979Iy&t=848"
- title: (none) -> Autonomous Torpedo Main Board
- moved on the sheet: A1, H1, H2, IC1, IC7, J5, J6

Commit message: feb23 updates
Parts:
- removed C12, C5: 0.1μF, Capacitor_SMD:C_0603_1608Metric, symbol Device:C
- removed C28, C29: 22nF, Capacitor_SMD:C_0603_1608Metric, symbol Device:C
- removed IC1: ICM-20948, SamacSys_Parts:QFN40P300X300X105-25N-D, symbol SamacSys_Parts:ICM-20948
- removed J7, J8: Conn_01x07, Connector_PinHeader_2.54mm:PinHeader_1x07_P2.54mm_Vertical, symbol Connector_Generic:Conn_01x07
- removed R12, R15, R16, R17: 10k, Resistor_SMD:R_0201_0603Metric, symbol Device:R
- removed S1: Scroll wheel encoder, switches_and_dials:EN10HT1212N5HH3, symbol switches dials and such:EN10HT1212N5HH3
- added A2: Grove AI Vision Module V2, board_board_connection:Grove conn, symbol board-connections:Grove-AI-Vision-Module-V2
- added C30: 1μF, symbol Device:C
- added C31, C32: 2.2μF, symbol Device:C
- added C33, C34: 0.1μF, symbol Device:C
- added C35: 220nF, symbol Device:C
- added H3: 22pin->15pin Adapter Slot, MountingEquipment:slot, symbol Mechanical:MountingHole
- added IC10: LIS2MDLTR: Magnetometer, LGA-12, symbol SamacSys_Parts:LIS2MDLTR
- added IC9: TPS60150DRVR: 3.3V->5V, SON65P200X200X80-7N, symbol SamacSys_Parts:TPS60150DRVR
- added U3: LSM6DSOTR: Acc+Gyro+Temp, LGA-14L_2P5X3X0P86_STM, symbol 2025-02-22_17-21-41:LSM6DSOTR
- added U4: ILPS22QS: Air Pressure+Temp, SamacSys_Parts:LPS22HHTR, symbol Sensor_Pressure:LPS25HB_1
- F1: value Fuse -> Fuse Holder
- IC7: value AP7362-33SP-13 -> AP7362-33SP-13: Batt->3.3V
- IC8: value TPS76918DBVR -> TPS76918DBVR: 3.3V->1.8V
- J5: footprint SamacSys_Parts:motor wire conn -> SamacSys_Parts:009276008021106
- J9: value UPIXEL Connector -> MTF-02P Connector
Connections:
- net +3.3V: now also A2.12 (3V3), C32.1, C33.1, C34.1, IC10.10 (VDD_IO), IC10.3 (CS), IC10.9 (VDD), IC9.2 (VIN), IC9.6 (ENA), U3.12 (CS), U3.5 (VDDIO), U3.8 (VDD), U4.1 (Vdd_IO), U4.10 (VDD), U4.6 (CS); no longer C23.1, IC7.5 (OUT_1), IC7.7 (OUT_3)
- net +BATT: no longer J9.1 (Pin_1)
- net GND: now also A2.13 (GND), C31.2, C32.2, C33.2, C34.2, C35.2, IC10.6 (GND_1), IC10.8 (GND_2), IC9.1 (GND), IC9.7 (EP), U3.6 (GND), U3.7 (GND), U4.3 (GND), U4.5 (AH2/QVAR2), U4.7 (AH1/QVAR1), U4.8 (GND), U4.9 (GND)
- net GROVE_DEBUG_LED1: now also A2.3 (D2/A2)
- net GROVE_RST: now also A2.4 (D3/A3)
- net IMU_INT: now also U3.4 (INT1)
- net SCL2: now also U3.13 (SCL), U4.2 (SCL)
- net SCL4: now also A2.6 (D5/SCL)
- net SDA2: now also U3.14 (SDA), U4.4 (SDA)
- net SDA4: now also A2.5 (D4/SDA)
- new net: IC10.4 (SDA/SDI/SDO), U3.2 (SDx)
- new net: IC10.1 (SCL/SPC), U3.3 (SCx)
- new net: C30.1, IC9.5 (CP-)
- new net: C30.2, IC9.4 (CP+)
- new net: C23.1, IC7.5 (OUT_1)
- new net: C35.1, IC10.5 (C1)
- new net +5V: C31.1, IC9.3 (VOUT), J9.1 (Pin_1)
- no-connect marks 40 -> 33
Other:
- note added: "IMU VDDIO Supply"
- note added: "Wired up in mode 2"
- moved on the sheet: C10, C11, F1, H1, H2

Commit message: flex_pcb_updates
Parts:
- removed C10: 1μF, Capacitor_SMD:C_0603_1608Metric, symbol Device:C
- removed C11: 2.2μF, Capacitor_SMD:C_0603_1608Metric, symbol Device:C
- removed IC8: TPS76918DBVR: 3.3V->1.8V, SamacSys_Parts:SOT95P280X145-5N, symbol SamacSys_Parts:TPS76918DBVR
Connections:
- net SDA_MAG: now reaches IC10.4 (SDA/SDI/SDO), U3.2 (SDx)
- net SCL_MAG: now reaches IC10.1 (SCL/SPC), U3.3 (SCx)
- no-connect marks 33 -> 32
Other:
- note removed: "0.2-2Ω ESR!!!"
- note removed: "IMU VDDIO Supply"

Commit message: everything is connected
Parts:
- removed F1: Fuse Holder, Capacitor_SMD:C_0603_1608Metric, symbol Device:Fuse
- removed J12: Conn_01x01, Connector_PinHeader_1.27mm:PinHeader_1x01_P1.27mm_Vertical, symbol Connector_Generic:Conn_01x01
- removed J13: Fan, Connector_PinSocket_1.27mm:PinSocket_1x02_P1.27mm_Vertical, symbol Connector_Generic:Conn_01x02
- removed J6: LiHV (3.8V), Connector_PinHeader_2.54mm:PinHeader_1x02_P2.54mm_Vertical, symbol Connector_Generic:Conn_01x02
- removed Q1, Q2: BSS138, Package_TO_SOT_SMD:SOT-23, symbol Transistor_FET:BSS138
- removed Q3: NMOS, symbol Simulation_SPICE:NMOS
- removed SW1: SW_SPDT, Connector_PinSocket_1.27mm:PinSocket_1x02_P1.27mm_Vertical, symbol Switch:SW_SPDT
- added C10, C11: 0.1μF, Capacitor_SMD:C_0603_1608Metric, symbol Device:C
- added C5: 1μF, Capacitor_SMD:C_0603_1608Metric, symbol Device:C
- added F2: Fuse Holder, SamacSys_Parts:0154001.DRT, symbol SamacSys_Parts:0154010.DR
- added H4: MountingHole, MountingHole:MountingHole_2.2mm_M2, symbol Mechanical:MountingHole
- added J13: I2C2 Access, SamacSys_Parts:BM04B-SRSS-TB_LFSN_, symbol Connector_Generic:Conn_01x04
- added J6: Batt+, Connector_PinHeader_2.54mm:PinHeader_1x01_P2.54mm_Vertical, symbol Connector_Generic:Conn_01x01
- added J7: Batt-, Connector_PinHeader_2.54mm:PinHeader_1x01_P2.54mm_Vertical, symbol Connector_Generic:Conn_01x01
- added J8: MTF-02P Connector, Connector_PinSocket_1.27mm:PinSocket_1x04_P1.27mm_Vertical, symbol Connector_Generic:Conn_01x04
- added Q5: DMG1013UW-7, SamacSys_Parts:2SC2712GRLF, symbol Simulation_SPICE:PMOS
- added Q6: PMOS SI4435FDY, SamacSys_Parts:SOIC127P600X175-8N, symbol Simulation_SPICE:PMOS
- added Q7: NMOS, SamacSys_Parts:SOTFL95P240X88-3N, symbol Simulation_SPICE:NMOS
- added R12, R15, R16, R17, R22: 10k, Resistor_SMD:R_0603_1608Metric, symbol Device:R
- added R23: 100k, Resistor_SMD:R_0603_1608Metric, symbol Device:R
- added S1: MSK12C02, SamacSys_Parts:MSK12C02, symbol SamacSys_Parts:MSK12C02
- added SW2, SW3, SW4: SW_SPST, SamacSys_Parts:436331045822, symbol Switch:SW_SPST
- added SW5: button, SamacSys_Parts:B3U3100PMB, symbol Switch:SW_MEC_5G
- A2: footprint board_board_connection:Grove conn -> board_board_connection:Grove conn_limited_pinout
- C24, C26: value ??μF -> 12μF
- C30, C31, C32, C33, C34, C35: footprint (none) -> Capacitor_SMD:C_0603_1608Metric
- D1: LCSC (none) -> C189306
- D2, D4: footprint Capacitor_SMD:C_0603_1608Metric -> LED_SMD:LED_0805_2012Metric; LCSC (none) -> C125103
- D3: footprint Capacitor_SMD:C_0603_1608Metric -> LED_SMD:LED_0805_2012Metric; LCSC (none) -> C284922
- H3: value 22pin->15pin Adapter Slot -> MountingHole; footprint MountingEquipment:slot -> MountingHole:MountingHole_2.2mm_M2
- IC10: footprint LGA-12 -> SamacSys_Parts:LGA-12
- IC9: footprint SON65P200X200X80-7N -> SamacSys_Parts:SON65P200X200X80-7N
- J10, J11: footprint Connector_PinSocket_2.00mm:PinSocket_2x02_P2.00mm_Vertical -> SamacSys_Parts:BM04B-SRSS-TB_LFSN_
- J9: value MTF-02P Connector -> I2C2 Access; footprint Connector_PinSocket_2.00mm:PinSocket_2x02_P2.00mm_Vertical -> SamacSys_Parts:BM04B-SRSS-TB_LFSN_
- R10: value R -> 260; footprint Resistor_SMD:R_0201_0603Metric -> Resistor_SMD:R_0603_1608Metric
- R11, R9: value R -> 100; footprint Resistor_SMD:R_0201_0603Metric -> Resistor_SMD:R_0603_1608Metric
- R13, R14, R5, R7, R8: footprint Resistor_SMD:R_0201_0603Metric -> Resistor_SMD:R_0603_1608Metric
- R18: value ??? -> 1.5k; footprint Resistor_SMD:R_0201_0603Metric -> Resistor_SMD:R_0603_1608Metric
- R6: value R -> 350; footprint Resistor_SMD:R_0201_0603Metric -> Resistor_SMD:R_0603_1608Metric
- U3: footprint LGA-14L_2P5X3X0P86_STM -> SamacSys_Parts:LGA-14L_2P5X3X0P86_STM
- Y2: value 32MHz? -> 16MHz; footprint (none) -> SamacSys_Parts:X322516MOB4SI
Connections:
- net +3.3V: now also C23.1, IC7.5 (OUT_1), IC7.7 (OUT_3), J9.1 (Pin_1), C11.1, Q5.3 (S), S1.A1 (NC), SW2.2 (B), SW3.2 (B), SW4.2 (B); no longer A1.12 (3V3), J10.1 (Pin_1)
- net +5V: now also J8.3 (Pin_3); no longer J9.1 (Pin_1)
- net +BATT: now also C5.2, Q6.5 (D), Q6.6 (D), Q6.7 (D), Q6.8 (D), R22.1
- net GND: now also C10.2, C11.2, J7.1 (Pin_1), J8.4 (Pin_4), Q7.3 (S), R12.1, R15.2, R16.2, R17.2, R23.1, S1.C1 (NO), S1.MP1, S1.MP2, S1.MP3, S1.MP4, SW5.1 (A)
- net HSE_OUT: now also C26.2, Y2.3; no longer R18.1
- net MOTOR0_IN: now also U2.10 (PA2); no longer U2.11 (PA3)
- net MOTOR0_PWM: now also U2.11 (PA3); no longer U2.10 (PA2)
- net MOTOR2_IN: now also U2.18 (PB1); no longer U2.22 (PB10)
- net MOTOR2_PWM: now also U2.22 (PB10); no longer U2.18 (PB1)
- net OPT_FLOW_RX: now also J8.1 (Pin_1); no longer J9.2 (Pin_2)
- net SCL2: now also J9.2 (Pin_2)
- net SDA2: now also J9.3 (Pin_3)
- net at R5.2: now also S1.B1 (COM)
- net at J10.2 (Pin_2): now also A1.7 (D6/TX); no longer A1.8 (D7/RX/SS)
- net at J10.3 (Pin_3): now also A1.8 (D7/RX/SS); no longer A1.7 (D6/TX)
- net at C30.1: now also IC9.4 (CP+); no longer IC9.5 (CP-)
- net at C30.2: now also IC9.5 (CP-); no longer IC9.4 (CP+)
- net ESP32_pmos_gate: now reaches A1.14 (VSUB)
- net ESP32_pmos_gate: now also Q5.2 (G), R12.2
- net STM32_PB5: now reaches U2.43 (PB5)
- net STM32_PB5: now also J13.2 (Pin_2)
- net FAN renamed STM32_PC13
- net INV_POWER_SHUTOFF renamed POWER_SHUTOFF
- net POWER_SHUTOFF: now also C10.1, Q7.2 (G), R22.2, R23.2
- net LIGHT: no longer names the net of J4.3
- net LIGHT_COMMS renamed STM32_PA11
- net STM32_PA11: now also J13.3 (Pin_3), J13.4 (Pin_4)
- net MODE_SEL_DIAL1 renamed MODE_SEL_UP
- net MODE_SEL_UP: now also R16.1, SW3.1 (A)
- net MODE_SEL_DIAL2 renamed MODE_SEL_DOWN
- net MODE_SEL_DOWN: now also R17.1, SW4.1 (A)
- net MODE_SEL_SWITCH renamed MODE_SEL_ENTER
- net MODE_SEL_ENTER: now also R15.1, SW2.1 (A)
- net OPT_FLOW_TX: no longer names the net of U2.44 (PB6)
- net OPT_FLOW_TX: no longer J9.3 (Pin_3)
- net UNUSED ADC renamed STM32_PB2
- net STM32_PB2: now also J13.1 (Pin_1)
- new net Batt_terminal+: F2.2, J6.1 (Pin_1)
- new net ESP32_3.3V: A1.12 (3V3), Q5.1 (D)
- new net NMOS_drain: Q6.4 (G), Q7.1 (D), R18.2, SW5.2 (B)
- new net PMOS_drain: C5.1, F2.1, Q6.1 (S), Q6.2 (S), Q6.3 (S), R18.1
- no-connect marks 32 -> 34
Other:
- note added: "Prevents the 3.3V connection when the ESP32 is plugged in"
- note added: "Should there be a resistor for the ESP32 input pins?"
- note added: "The Grove AI Vision Module must be removed to be programmed"
- note added: "Unused ADC"
- note added: "Unused GPIO"
- note added: "unused TX for optical flow"
- note removed: "Grove AI Module V2 Connection"
- moved on the sheet: A1, A2, C22, C23, C24, C26, C27, C30, C31, C32, D1, D2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
