File: torpedo_pcbs/Grove_based_board/Grove_based_board.kicad_sch (KiCad schematic)
At the start: 81 parts, among them IC10 LIS2MDLTR: Magnetometer, IC6 VEML6040A3OG, IC7 AP7362-33SP-13: Batt->3.3V, IC9 TPS60150DRVR: 3.3V->5V, J1 503480-2200, J10 UART Comms, J11 LCD Screen, J13 I2C2 Access, J2 503480-2200, J3 503480-0440, J4 503480-0440, J5 Push-in Terminals, J6 Batt+, J7 Batt-, J8 MTF-02P Connector, J9 I2C2 Access, Q5 DMG1013UW-7, Q6 PMOS SI4435FDY, Q7 NMOS, SW2 SW_SPST, SW3 SW_SPST, SW4 SW_SPST, SW5 button, U1 STLINK-V3MINIE Edge Connector, U2 STM32G473CBU6, U3 LSM6DSOTR: Acc+Gyro+Temp, U4 ILPS22QS: Air Pressure+Temp, Y2 16MHz

Commit message: June-1-2025 jlcpcb order
Parts:
- removed C35: 220nF, Capacitor_SMD:C_0603_1608Metric, symbol Device:C
- removed IC10: LIS2MDLTR: Magnetometer, SamacSys_Parts:LGA-12, symbol SamacSys_Parts:LIS2MDLTR
- removed J1, J2: 503480-2200, SamacSys_Parts:5034802200, symbol SamacSys_Parts:503480-2200
- removed J10: UART Comms, SamacSys_Parts:BM04B-SRSS-TB_LFSN_, symbol Connector_Generic:Conn_01x04
- removed J11: LCD Screen, SamacSys_Parts:BM04B-SRSS-TB_LFSN_, symbol Connector_Generic:Conn_01x04
- removed J3, J4: 503480-0440, SamacSys_Parts:5034800440, symbol SamacSys_Parts:503480-0440
- removed J5: Push-in Terminals, SamacSys_Parts:009276008021106, symbol SamacSys_Parts:S8B-EH
- removed J9: I2C2 Access, SamacSys_Parts:BM04B-SRSS-TB_LFSN_, symbol Connector_Generic:Conn_01x04
- removed Q5: DMG1013UW-7, SamacSys_Parts:2SC2712GRLF, symbol Simulation_SPICE:PMOS
- removed S1: MSK12C02, SamacSys_Parts:MSK12C02, symbol SamacSys_Parts:MSK12C02
- removed U2: STM32G473CBU6, Package_DFN_QFN:QFN-48-1EP_7x7mm_P0.5mm_EP5.6x5.6mm, symbol MCU_ST_STM32G4:STM32G473CBUx
- removed U3: LSM6DSOTR: Acc+Gyro+Temp, SamacSys_Parts:LGA-14L_2P5X3X0P86_STM, symbol 2025-02-22_17-21-41:LSM6DSOTR
- added C12: 10μF, Capacitor_SMD:C_0603_1608Metric, symbol Device:C
- added C28: 1μF, Capacitor_SMD:C_0603_1608Metric, symbol Device:C
- added C29: 0.1μF, Capacitor_SMD:C_0603_1608Metric, symbol Device:C
- added IC1: ICM-42688-P, IIM42352, symbol SamacSys_Parts:ICM-42688-P
- added IC8: MMC5983MA-B, MMC5983MAB, symbol SamacSys_Parts:MMC5983MA-B
- added J1, J2: FH34SRJ-22S-0.5SH_99_, FH34SRJ22S05SH99, symbol SamacSys_Parts:FH34SRJ-22S-0.5SH_99_
- added J10: 1770940, SamacSys_Parts:1770940, symbol SamacSys_Parts:1770940
- added J11: I2C2 Access, SamacSys_Parts:BM04B-SRSS-TB_LFSN_, symbol Connector_Generic:Conn_01x06
- added J14, J9: LCD Screen, SamacSys_Parts:BM04B-SRSS-TB_LFSN_, symbol Connector_Generic:Conn_01x06
- added J3, J4: FH34SRJ-4S-0.5SH_50_, FH34SRJ4S05SH50, symbol SamacSys_Parts:FH34SRJ-4S-0.5SH_50_
- added J5: Conn_01x01, Connector_PinHeader_1.00mm:PinHeader_1x01_P1.00mm_Vertical, symbol Connector_Generic:Conn_01x01
- added Q1: SI1967DH-T1-GE3, SOT65P210X110-6N, symbol SamacSys_Parts:SI1967DH-T1-GE3
- added R19: 10k, Resistor_SMD:R_0603_1608Metric, symbol Device:R
- added SW1: button, SamacSys_Parts:B3U3100PMB, symbol Switch:SW_MEC_5G
- added TH1: 10k, Resistor_SMD:R_1206_3216Metric, symbol Device:Thermistor_NTC
- added U2: STM32G431CBUx, Package_DFN_QFN:QFN-48-1EP_7x7mm_P0.5mm_EP5.6x5.6mm, symbol MCU_ST_STM32G4:STM32G431CBUx
- C10, C11, C14, C15, C16, C17, C21, C27: LCSC (none) -> C14663
- C13, C22, C23: LCSC (none) -> C19702
- C18, C20, C25, C5: LCSC (none) -> C15849
- C19: LCSC (none) -> C57112
- C24, C26: value 12μF -> 12pF; LCSC (none) -> C38523
- C30: value 1μF -> 2.2μF; LCSC (none) -> C23630
- C31, C32: LCSC (none) -> C23630
- C33: value 0.1μF -> 2.2μF; LCSC (none) -> C23630
- C34: value 0.1μF -> 10nF; LCSC (none) -> C57112
- D1: footprint Capacitor_SMD:C_0603_1608Metric -> LED_SMD:LED_0805_2012Metric; LCSC C189306 -> C2286
- D2, D4: LCSC C125103 -> C2286
- D3: LCSC C284922 -> C2286
- F2: LCSC (none) -> C206909
- FB1: value FerriteBead -> 120R; LCSC (none) -> C22787
- IC7: LCSC (none) -> C780775
- IC9: LCSC (none) -> C182429
- J13: value I2C2 Access -> GPIO Access; footprint SamacSys_Parts:BM04B-SRSS-TB_LFSN_ -> Connector_PinHeader_1.27mm:PinHeader_1x04_P1.27mm_Vertical
- Q6: value PMOS SI4435FDY -> PMOS; LCSC (none) -> C67287
- Q7: LCSC (none) -> C10488
- R10: value 260 -> 200; LCSC (none) -> C8218
- R11, R9: value 100 -> 200; LCSC (none) -> C8218
- R12, R14, R15, R16, R17, R22: LCSC (none) -> C25804
- R13: LCSC (none) -> C4184
- R18: LCSC (none) -> C22843
- R23: LCSC (none) -> C14675
- R5: value 10k -> 1.5k; LCSC (none) -> C22843
- R6: value 350 -> 200; LCSC (none) -> C8218
- R7, R8: LCSC (none) -> C4190
- SW5: LCSC (none) -> C4364828
- Y2: LCSC (none) -> C12668
Connections:
- net BOOT0_STM is gone; now on net STM32_NRST: R5.1
- net ESP32_pmos_gate is gone; now on net ESP32PowGate: A1.14 (VSUB), R12.2
- net +3.3V: now also C28.2, C29.1, IC1.1 (AP_SDO_/_AP_AD0), IC1.12 (AP_CS), IC1.5 (VDDIO), IC1.8 (VDD), IC8.13 (VDDIO), IC8.2 (VDD), IC8.4 (SPI_CS), J11.1 (Pin_1), J14.1 (Pin_1), J3.3, J4.1, Q1.1 (S1), U2.1 (VBAT), U2.23 (VDD), U2.35 (VDD), U2.48 (VDD)
- net +3.3VA: now also R19.1, U2.20 (VREF+), U2.21 (VDDA)
- net BATT_ADC: now also U2.24 (PB11)
- net ESP32_3.3V: now also Q1.4 (S2)
- net GND: now also C12.2, C28.1, C29.2, IC1.11 (RESV_5), IC1.6 (GND), IC1.7 (RESV_3), IC1.9 (INT2_/_FSYNC_/_CLKIN), IC8.11 (GND_2), IC8.9 (GND_1), J1.MP1, J1.MP2, J11.4 (Pin_4), J11.5 (Pin_5), J11.6 (Pin_6), J14.4 (Pin_4), J14.5 (Pin_5), J14.6 (Pin_6), J2.MP1, J2.MP2, J3.4, J3.5 (MP1), J3.6 (MP2), J4.2, J4.5 (MP1), J4.6 (MP2), J9.4 (Pin_4), J9.5 (Pin_5), J9.6 (Pin_6), SW1.1 (A), TH1.2, U2.49 (VSS)
- net GPIO1: now also J4.3, U2.33 (PA11)
- net HSE_IN: now also U2.5 (PF0)
- net HSE_OUT: now also U2.6 (PF1)
- net JTCK: now also U2.37 (PA14)
- net JTDI: now also U2.38 (PA15)
- net JTDO: now also U2.41 (PB3)
- net JTMS: now also U2.36 (PA13)
- net JTRST: now also U2.42 (PB4)
- net MOTOR0_GAINSEL: now also U2.9 (PA1)
- net MOTOR0_IN: now also U2.10 (PA2)
- net MOTOR0_IPROPI: now also U2.8 (PA0)
- net MOTOR0_PWM: now also U2.11 (PA3)
- net MOTOR1_GAINSEL: now also U2.14 (PA6)
- net MOTOR1_IN: now also U2.15 (PA7)
- net MOTOR1_IPROPI: now also U2.12 (PA4)
- net MOTOR1_PWM: now also U2.13 (PA5)
- net MOTOR2_GAINSEL: now also U2.17 (PB0)
- net MOTOR2_IN: now also U2.18 (PB1)
- net MOTOR2_IPROPI: now also U2.16 (PC4)
- net MOTOR2_PWM: now also U2.22 (PB10)
- net MOTOR3_GAINSEL: now also U2.26 (PB13)
- net MOTOR3_IN: now also U2.25 (PB12)
- net MOTOR3_IPROPI: now also U2.28 (PB15)
- net MOTOR3_PWM: now also U2.27 (PB14)
- net Motor driver0/OUT1: now also J10.1 (1.1), J10.2 (1.2)
- net Motor driver0/OUT2: now also J10.3 (2.1), J10.4 (2.2)
- net Motor driver1/OUT1: now also J10.5 (3.1), J10.6 (3.2)
- net Motor driver1/OUT2: now also J10.7 (4.1), J10.8 (4.2)
- net Motor driver2/OUT1: now also J10.10 (5.2), J10.9 (5.1)
- net Motor driver2/OUT2: now also J10.11 (6.1), J10.12 (6.2)
- net Motor driver3/OUT1: now also J10.13 (7.1), J10.14 (7.2)
- net Motor driver3/OUT2: now also J10.15 (8.1), J10.16 (8.2)
- net OPT_FLOW_RX: now also U2.32 (PA10)
- net POWER_SHUTOFF: now also U2.4 (PC15)
- net SCL2: now also R8.2, IC1.13 (AP_SCL_/_AP_SCLK), IC8.1 (SCL/SPI_SCK), J11.2 (Pin_2), J3.1, U2.31 (PA9); no longer R7.2
- net SCL4: now also J14.2 (Pin_2), U2.46 (PB8)
- net SDA2: now also R7.2, IC1.14 (AP_SDA_/_AP_SDIO_/_AP_SDI), IC8.16 (SDA/SPI_SDI), J11.3 (Pin_3), J3.2, U2.30 (PA8); no longer R8.2
- net SDA4: now also J14.3 (Pin_3), U2.45 (PB7)
- net STM32_DEBUG_LED1: now also U2.47 (PB9)
- net STM32_NRST: no longer C21.2
- net STM32_PB5: now also U2.43 (PB5)
- net STM32_PC13: now also J13.3 (Pin_3), U2.2 (PC13)
- net XSHUT: now also J4.4, U2.34 (PA12)
- net at R5.2: now also C21.2, SW1.2 (B), U2.7 (PG10)
- net at A1.7 (D6/TX): now also J9.2 (Pin_2)
- net at A1.8 (D7/RX/SS): now also J9.3 (Pin_3)
- net ESP32PowGate: now reaches A1.14 (VSUB)
- net ESP32PowGate: now also Q1.2 (G1), Q1.5 (G2)
- net PMOS_drain renamed PMOS_source
- net RX renamed TX_STLINK
- net TX_STLINK: now also U2.39 (PC10)
- net STM32_PA11 renamed STM32_PC14
- net STM32_PC14: now also U2.3 (PC14); no longer J13.3 (Pin_3)
- net STM32_PB2: no longer names the net of J13.1 (Pin_1)
- net TX renamed RX_STLINK
- net RX_STLINK: now also U2.40 (PC11)
- new net: J1.1, J2.22
- new net: J1.10, J2.13
- new net: J1.11, J2.12
- new net: J1.12, J2.11
- new net: J1.13, J2.10
- new net: J1.14, J2.9
- new net: J1.15, J2.8
- new net: J1.16, J2.7
- new net: J1.17, J2.6
- new net: J1.18, J2.5
- new net: J1.19, J2.4
- new net: J1.2, J2.21
- new net: J1.20, J2.3
- new net: J1.21, J2.2
- new net: J1.22, J2.1
- new net: J1.3, J2.20
- new net: J1.4, J2.19
- new net: J1.5, J2.18
- new net: J1.6, J2.17
- new net: J1.7, J2.16
- new net: J1.8, J2.15
- new net: J1.9, J2.14
- new net: Q1.3 (D2), Q1.6 (D1)
- new net: IC8.15 (INT), J5.1 (Pin_1)
- new net Batt_temp: R19.2, TH1.1, U2.19 (PB2)
- new net IMU_int: IC1.4 (INT1_/_INT), U2.29 (PC6)
- new net MMC5983MA_Cap: C12.1, IC8.10 (CAP)
- no-connect marks 34 -> 36
Other:
- note added: "JTAG doesn't need BOOT0"
- note removed: "Should there be a resistor for the ESP32 input pins?"
- note removed: "Unused ADC"
- note removed: "Wired up in mode 2"
- moved on the sheet: A1, C13, C14, C15, C16, C17, C21, C24, C26, D4, J7, R10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
