File: torpedo_pcbs/Grove_based_board/motor_driver.kicad_sch (KiCad schematic)
At the start: 4 parts, among them IC2 DRV8213DSGR

Commit message: June-1-2025 jlcpcb order
Parts:
- C1: LCSC (none) -> C14663
- C6: LCSC (none) -> C178330
- IC2: LCSC (none) -> C22407186
- R2: footprint Resistor_SMD:R_0805_2012Metric -> Resistor_SMD:R_0603_1608Metric; LCSC (none) -> C14892
Changed lines of the file:
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@@
 			)
 		)
-		(property "Footprint" "Resistor_SMD:R_0805_2012Metric"
+		(property "Footprint" "Resistor_SMD:R_0603_1608Metric"
 			(at 187.452 90.17 90)
 			(effects
@@
 			)
 		)
-		(property "Datasheet" "~"
+		(property "Datasheet" "https://jlcpcb.com/partdetail/15564-0603WAF8451T5E/C14892"
 			(at 189.23 90.17 0)
 			(effects
@@
 			)
 		)
-		(property "LCSC" ""
+		(property "LCSC" "C14892"
 			(at 189.23 90.17 0)
 			(effects
@@
 			)
 		)
-		(property "LCSC" ""
+		(property "LCSC" "C178330"
 			(at 110.49 87.63 0)
 			(effects
@@
 			)
 		)
-		(property "LCSC" ""
+		(property "LCSC" "C14663"
 			(at 123.825 87.63 0)
 			(effects
@@
 		(on_board yes)
 		(dnp no)
-		(fields_autoplaced yes)
 		(property "Reference" "IC2"
 			(at 152.4 76.2 0)
@@
 			)
 		)
-		(property "LCSC" ""
+		(property "LCSC" "C22407186"
 			(at 134.62 83.82 0)
 			(effects
